File: PCB/H30_controler_board.kicad_sch (KiCad schematic)
At the start: 41 parts, among them IC1 LTC4359IMS8#PBF, IC2 MP2338GTL-P, J1 Conn_01x02_Socket, Q1 PSMNR56-25YLEX, Q10 XT60_YELLOW, Q11 XT60_YELLOW, Q2 PSMNR56-25YLEX, Q3 PSMNR56-25YLEX, Q4 PSMNR56-25YLEX, Q5 PSMNR56-25YLEX, Q6 PSMNR56-25YLEX, Q7 SI2301-TP, Q8 SI2301-TP, Q9 SI2301-TP, U3 STM32L476RCTx

Commit message: Add files via upload
Parts:
- added C7, C8: C_Polarized, symbol Device:C_Polarized
- added D4: SMAT70A-13-F, SMAT70A-13-F:DIOM5226X230N, symbol SMAT70A-13-F:SMAT70A-13-F
- added D5: SMAJ24A, SMAJ24A:DIOM4325X250N, symbol SMAJ24A:SMAJ24A
- added D6, D7: B240A-E3_5AT, B240A-E3_5AT:DIOM5127X229N, symbol B240A-E3_5AT:B240A-E3_5AT
- added Q12: SI2301-TP, SI2301:SOT95P237X125-3N, symbol SI2301-TP:SI2301-TP
- added Q13: PSMNR56-25YLEX, PSMNR56-25YLEX:PSMNR5830YLHX, symbol PSMNR56-25YLEX:PSMNR56-25YLEX
- added R16: 100K, Resistor_SMD:R_0603_1608Metric, symbol Device:R
- added R17: 2.2K, Resistor_SMD:R_0603_1608Metric, symbol Device:R
- added R18: 0.1R, Resistor_SMD:R_0603_1608Metric, symbol Device:R
- added R19, R20: ?, Resistor_SMD:R_0603_1608Metric, symbol Device:R
- added R22, R23, R24, R25, R27: 10K, Resistor_SMD:R_0603_1608Metric, symbol Device:R
- added R26: 220R, Resistor_SMD:R_0603_1608Metric, symbol Device:R
- added SW2: SW_Nidec_CAS-120A1, 0S102011MA1QN1C:0S102011MA1QN1C, symbol Switch:SW_Nidec_CAS-120A1
- D3: footprint (none) -> LED_SMD:LED_0603_1608Metric
- L1: footprint (none) -> 7443340680:WE-HCC_807021
- R15: value 5K -> ?
- R2: value 100K -> 10K
Connections:
- net +H30: now also R2.2, D4.C, R24.1
- net -H30: now also R17.1, R22.2, R23.2; no longer R15.1, R2.2
- net EN: now also R17.2; no longer R15.2
- net Gate_Q3_Q4: no longer R2.1
- net LIPO+: now also C7.1, C8.1
- net LIPO-: now also R15.2, Q13.1 (S), Q13.2 (S), Q13.3 (S), R16.2, R19.2, R20.2, R25.2, R27.1
- net ST_H30_LIPO: now also R23.1
- net ST_ShortCUT: now also R22.1
- net at C1.2, IC1.6 (VSS), R1.1: now also D5.C
- net at Q6.1 (S): now also Q6.2 (S), Q6.3 (S), R15.1, R19.1, R20.1
- net at Q6.4 (G): now also R26.2
- net Capa_out: now reaches Q6.5 (D)
- new net: D6.2 (A), R18.1
- new net: Q12.3 (D), R26.1, R27.2
- new net: Q13.4 (G), R16.1, R2.1
- new net: R25.1, SW2.3 (A)
- new net: D4.A, D5.A
- new net: D6.1 (K), D7.1 (K), Q12.2 (S), SW2.1 (C)
- new net: Q12.1 (G), SW2.2 (B)
- new net: D7.2 (A), R24.2
- new net capa_out: C7.2, C8.2, Q13.5 (D), R18.2
Other:
- note added: "24V"
- note added: "70V"
- note added: "Nmos car Rds(on) <<"
- note added: "Pas de fonction d'arret SHDN 2.6uA"
- note added: "Vgsth = -0.45"
- note added: "Vgsth = 1.2"
- note added: "batt plug = capa connected batt out = capa disconnected"
- note added: "dimentionnement res"
- note added: "dimnetionner reistance de decharge"
- note added: "open drain Pin 5V tolerant"
- note removed: "3V3 on only when H30 > Vmin LDO else pull down"
- note removed: "Attention si pas 3.3V etat flotant..."
- note removed: "DIODE ?"
- note removed: "N mos car Rds(on) <<"
- note removed: "batterie → interrupteur (MOSFET) → circuit → capas (isolées)"
- note removed: "open drain"
- note removed: "switch de decharge"
- moved on the sheet: D2, J1, L1, Q7, R3, R6, R7, U3

Commit message: Add files via upload
Parts:
- removed D1, D6, D7: B240A-E3_5AT, B240A-E3_5AT:DIOM5127X229N, symbol B240A-E3_5AT:B240A-E3_5AT
- removed J1: Conn_01x02_Socket, Connector_PinSocket_2.54mm:PinSocket_1x02_P2.54mm_Vertical, symbol Connector:Conn_01x02_Socket
- added C1, C3: 1uF, Capacitor_SMD:C_0603_1608Metric, symbol Device:C
- added C13: 4.7uF, Capacitor_SMD:C_0603_1608Metric, symbol Device:C_Small
- added C14, C15, C16, C17, C18, C23: 100nf, Capacitor_SMD:C_0603_1608Metric, symbol Device:C_Small
- added C19: 1uF, Capacitor_SMD:C_0603_1608Metric, symbol Device:C_Small
- added C2, C4: 100nF, Capacitor_SMD:C_0603_1608Metric, symbol Device:C
- added C20: 10nF, Capacitor_SMD:C_0603_1608Metric, symbol Device:C_Small
- added C21, C22: 7.2pF, Capacitor_SMD:C_0603_1608Metric, symbol Device:C_Small
- added C212, C213: 100n, Capacitor_SMD:C_0603_1608Metric, symbol Device:C_Small
- added C24: 220uF, symbol Device:C_Polarized
- added C65: 0.1uF, Capacitor_SMD:C_0603_1608Metric, symbol Device:C
- added D1, D11, D6, D7, D9: STPS2L30A, STPS2L30A:DIOM5126X265N, symbol STPS2L30A:STPS2L30A
- added D10: RED, LED_SMD:LED_0603_1608Metric, symbol Device:LED
- added D12: BLUE, LED_SMD:LED_0603_1608Metric, symbol Device:LED
- added D201: 19-237/R6GHBHC-A01/2T, 19-237_R6GHBHC-A01_2T:19237R6GHBHCA012T, symbol Device:LED_RGBA
- added D5: GREEN, LED_SMD:LED_0603_1608Metric, symbol Device:LED
- added F1: MF-MSMF200_12X-2, MF-MSMF200_12X-2:MFMSMF20012X2, symbol MF-MSMF200_12X-2:MF-MSMF200_12X-2
- added FB200: 600 @ 600 MHz, Inductor_SMD:L_0805_2012Metric, symbol Device:Ferrite_Bead_Small
- added H1, H2, H3, H4: MountingHole_Pad, MountingHole:MountingHole_3.2mm_M3_Pad_Via, symbol Mechanical:MountingHole_Pad
- added IC3: W25N01GVZEIG, W25N01GVZEIG:SON127P800X600X80-9N-D, symbol W25N01GVZEIG:W25N01GVZEIG
- added J1, J3, J4, J5, J6, J8: 62000411622, Connector_THT_Wurth:J_Wurth_WR-WTB_62000411622, symbol Connector_Wurth_WR-WTB:62000411622
- added J10, J2, J9: 62000211622, Connector_THT_Wurth:J_Wurth_WR-WTB_62000211622, symbol Connector_Wurth_WR-WTB:62000211622
- added J12: USB_C_Receptacle_USB2.0_14P, USBC:USBC, symbol Connector:USB_C_Receptacle_USB2.0_14P
- added J401: SWD, Connector_PinHeader_1.27mm:PinHeader_2x05_P1.27mm_Vertical_SMD, symbol Connector_Generic:Conn_02x05_Odd_Even
- added J7: 62000611622, Connector_THT_Wurth:J_Wurth_WR-WTB_62000611622, symbol Connector_Wurth_WR-WTB:62000611622
- added JP1, JP2: ~, jumper_footprints:Jumper_0603, symbol My_Jumper:jumper_close
- added PS1: LD39050PU33R, LD39050PU33R:SON95P300X300X100-7N-D, symbol LD39050PU33R:LD39050PU33R
- added Q14: AO3401A, Package_TO_SOT_SMD:SOT-23, symbol Transistor_FET:AO3401A
- added R11: 2.2K, Resistor_SMD:R_0603_1608Metric, symbol Device:R
- added R206, R207, R208: 1k, Resistor_SMD:R_0603_1608Metric, symbol Device:R_Small
- added R28, R32: 10K, Resistor_SMD:R_0603_1608Metric, symbol Device:R_Small
- added R29: 47R, Resistor_SMD:R_0603_1608Metric, symbol Device:R_Small
- added R30, R31: 2K2, Resistor_SMD:R_0603_1608Metric, symbol Device:R_Small
- added R33, R35: 5K1, Resistor_SMD:R_0603_1608Metric, symbol Device:R
- added R34, R36, R37, R38, R39, R40, R400, R401, R402, R403, R41, R42, R43, R44, R45, R46: 22, Resistor_SMD:R_0603_1608Metric, symbol Device:R_Small
- added R48: 2k2, Resistor_SMD:R_0603_1608Metric, symbol Device:R_Small
- added SW2: SW_Nidec_CAS-120A1, 450404015514:450404015514, symbol Switch:SW_Nidec_CAS-120A1
- added SW4: ~, SKSGPAE010:SKSG, symbol SKSGPAE010_V2:SKSGPAE010
- added TP1: V_USB, TestPoint:TestPoint_Pad_D2.0mm, symbol Connector:TestPoint
- added U9: USBLC6-2SC6, Package_TO_SOT_SMD:SOT-23-6, symbol Power_Protection:USBLC6-2SC6
- added Y1: 16MHz, NX3225SA-16.000000MHZ-B3:NX3225SA16000000MHZB3, symbol Device:Crystal_GND24_Small
- D2: renamed from D3; value LED -> RED
- L1: footprint 7443340680:WE-HCC_807021 -> SRP5020CC-6R8M:INDPM5752X200N
- R1: renamed from R12; value 10K -> 100K
- SW1: renamed from SW2; footprint 0S102011MA1QN1C:0S102011MA1QN1C -> 450404015514:450404015514
- renumbered C1 to C10, C7 to C11, C8 to C12, C2 to C5, C3 to C6, C6 to C7, C4 to C8, C5 to C9, D4 to D3, D5 to D4, D2 to D8, IC2 to IC1, IC1 to IC2, Q10 to Q1, Q12 to Q10, Q6 to Q11, Q7 to Q12, Q11 to Q13, Q8 to Q2, Q5 to Q3, Q1 to Q4, Q2 to Q5, Q9 to Q6, Q3 to Q7, Q4 to Q8, Q13 to Q9, R13 to R10, R1 to R12, R23 to R13, R8 to R14, R5 to R15, R24 to R16, R25 to R17, R2 to R18, R18 to R19, R14 to R2, R16 to R20, R27 to R21, R26 to R22, R20 to R23, R15 to R24, R3 to R25, R19 to R26, R6 to R27, R17 to R3, R22 to R4, R7 to R5, R4 to R6, R9 to R7, R10 to R8, R11 to R9, U3 to U1
Connections:
- net ST_EV is gone; now on net TIM3_CH1: R25.2, R27.1
- net ST_H30_LIPO is gone; now on net TIM3_CH3: R13.1, R14.1
- net ST_ShortCUT is gone; now on net TIM1_CH1: R4.1, R5.1
- net +12V: now also D1.1 (K), F1.1; no longer C5.1, IC1.2 (VIN), R2.2
- net +3V3: now also U1.1 (VBAT), U1.19 (VDD), U1.32 (VDD), U1.48 (VDDUSB), U1.64 (VDD), C13.1, C14.1, C15.1, C16.1, C17.1, C18.1, C212.1, C213.1, C3.1, C4.1, D201.4 (A), FB200.2, IC3.8 (VCC), J1.4, J3.4, J4.4, J401.1 (Pin_1), J5.4, J6.4, J7.6, J8.4, PS1.4 (VOUT), R30.2, R31.2, SW2.1 (C)
- net +5V: now also C1.1, C2.1, D11.1 (K), D12.2 (A), J10.2, J9.2, PS1.1 (EN), PS1.6 (VIN), R11.2
- net +H30: now also D1.2 (A)
- net -H30: now also C24.2, D5.1 (K), H1.1, H2.1, H3.1, H4.1, J2.1, Q14.1 (G)
- net -ST: now also U1.12 (VSSA), U1.18 (VSS), U1.31 (VSS), U1.47 (VSS), U1.63 (VSS), C1.2, C13.2, C14.2, C15.2, C16.2, C17.2, C18.2, C19.2, C2.2, C20.2, C21.2, C212.2, C213.2, C22.2, C23.2, C3.2, C4.2, C65.2, D10.1 (K), IC3.4 (GND), IC3.9 (EP), J1.1, J10.1, J12.A1 (GND), J12.A12 (GND), J12.B1 (GND), J12.B12 (GND), J3.1, J4.1, J401.3 (Pin_3), J401.5 (Pin_5), J401.9 (Pin_9), J5.1, J6.1, J7.1, J8.1, J9.1, PS1.2 (GND), PS1.7 (PAD), SW2.3 (A), SW4.2, SW4.4, SW4.5, SW4.6, U9.2 (GND), Y1.2, Y1.4
- net at R19.1: now also D7.2 (A)
- net ADC3_IN3+: now reaches U1.10 (PC2)
- net ADC3_IN3+: now also R37.2
- net ADC3_IN4-: now reaches U1.11 (PC3)
- net ADC3_IN4-: now also R38.2
- net +3V3A: now reaches U1.13 (VDDA)
- net +3V3A: now also C19.1, C20.1, FB200.1
- net UART4_TX: now reaches U1.14 (PA0)
- net UART4_TX: now also R46.2
- net UART4_RX: now reaches U1.15 (PA1)
- net UART4_RX: now also R45.2
- net TIM2_CH3: now reaches U1.16 (PA2)
- net TIM2_CH3: now also R207.1
- net TIM2_CH4: now reaches U1.17 (PA3)
- net TIM2_CH4: now also R208.2
- net SPI1_CS: now reaches U1.2 (PC13)
- net SPI1_CS: now also J7.5
- net SPI1_SCK: now reaches U1.21 (PA5)
- net SPI1_SCK: now also J7.2
- net QUADSPI_IO3: now reaches U1.22 (PA6)
- net QUADSPI_IO3: now also IC3.7 (~{HOLD_(IO3_)})
- net QUADSPI_IO2: now reaches U1.23 (PA7)
- net QUADSPI_IO2: now also IC3.3 (~{WP_(IO2_)})
- net USART3_TX: now reaches U1.24 (PC4)
- net USART3_TX: now also R44.2
- net USART3_RX: now reaches U1.25 (PC5)
- net USART3_RX: now also R43.2
- net QUADSPI_IO1: now reaches U1.26 (PB0)
- net QUADSPI_IO1: now also IC3.2 (DO_(IO1_))
- net QUADSPI_IO0: now reaches U1.27 (PB1)
- net QUADSPI_IO0: now also IC3.5 (DI_(IO0_))
- net QUADSPI_CSK: now reaches U1.29 (PB10)
- net QUADSPI_CSK: now also IC3.6 (CLK)
- net QUADSPI_NCS: now reaches U1.30 (PB11)
- net QUADSPI_NCS: now also IC3.1 (~{CS})
- net TIM3_CH1: now reaches U1.37 (PC6)
- net TIM3_CH1: now also R48.2
- net TIM3_CH3: now reaches U1.39 (PC8)
- net TIM1_CH1: now reaches U1.41 (PA8)
- net JP-: now reaches U1.44 (PA11)
- net JP-: now also JP1.1
- net JP+: now reaches U1.45 (PA12)
- net JP+: now also JP2.1
- net SWDIO: now reaches U1.46 (PA13)
- net SWDIO: now also R400.1
- net SWCLK: now reaches U1.49 (PA14)
- net SWCLK: now also R401.1
- net HSE_IN: now reaches U1.5 (PH0)
- net HSE_IN: now also C21.1, Y1.1
- net TIM2_CH1: now reaches U1.50 (PA15)
- net TIM2_CH1: now also R206.2
- net SWO: now reaches U1.55 (PB3)
- net SWO: now also R402.1
- net SPI1_MISO: now reaches U1.56 (PB4)
- net SPI1_MISO: now also J7.3
- net SPI1_MOSI: now reaches U1.57 (PB5)
- net SPI1_MOSI: now also J7.4
- net I2C1_SCL: now reaches U1.58 (PB6)
- net I2C1_SCL: now also R30.1, R40.2, R42.2
- net I2C1_SCA: now reaches U1.59 (PB7)
- net I2C1_SCA: now also R31.1, R39.2, R41.2
- net HSE_OUT: now reaches U1.6 (PH1)
- net HSE_OUT: now also R29.2
- net BOOT0: now reaches U1.60 (BOOT0)
- net BOOT0: now also R28.2
- net NRST: now reaches U1.7 (NRST)
- net NRST: now also C23.1, R403.1, SW4.1, SW4.3
- net ADC1_IN1+: now reaches U1.8 (PC0)
- net ADC1_IN1+: now also R34.2
- net ADC1_IN2-: now reaches U1.9 (PC1)
- net ADC1_IN2-: now also R36.2
- net at D8.1 (K), Q12.3 (D): now also J2.2
- net at Q10.2 (S), SW1.1 (C): now also D6.1 (K), D7.1 (K)
- net at R16.2: now also D6.2 (A)
- net Gate_Q3_Q4 renamed Gate_H30-OUT-
- net LIPO+ renamed OUT+
- net LIPO- renamed OUT-
- new net: D201.1 (RK), R206.1
- new net: D201.2 (GK), R207.2
- new net: D201.3 (BK), R208.1
- new net: J401.10 (Pin_10), R403.2
- new net: J401.2 (Pin_2), R400.2
- new net: J401.4 (Pin_4), R401.2
- new net: J401.6 (Pin_6), R402.2
- new net: J3.2, R40.1
- new net: J3.3, R39.1
- new net: C24.1, C5.1, D9.1 (K), IC1.2 (VIN), Q14.2 (S), R2.2
- new net: J8.2, R38.1
- new net: J5.2, R46.1
- new net: J5.3, R45.1
- new net: J12.A5 (CC1), R35.2
- new net: R28.1, R32.2, SW2.2 (B)
- new net: D12.1 (K), R48.1
- new net: J6.2, R42.1
- new net: J12.B5 (CC2), R33.2
- new net: D10.2 (A), R32.1
- new net: J1.2, R36.1
- new net: J1.3, R34.1
- new net: J6.3, R41.1
- new net: C22.1, R29.1, Y1.3
- new net: J8.3, R37.1
- new net: D5.2 (A), R11.1
- new net: F1.2, Q14.3 (D)
- new net: J4.3, R43.1
- new net: J4.2, R44.1
- new net +VBUS: C65.1, D11.2 (A), D9.2 (A), J12.A4 (VBUS), J12.A9 (VBUS), J12.B4 (VBUS), J12.B9 (VBUS), TP1.1, U9.5 (VBUS)
- new net GND: R33.1, R35.1
- new net USB_D+: J12.A6 (D+), J12.B6 (D+), JP2.2, U9.3 (I/O2), U9.4 (I/O2)
- new net USB_D-: J12.A7 (D-), J12.B7 (D-), JP1.2, U9.1 (I/O1), U9.6 (I/O1)
- no-connect marks 3 -> 9
Other:
- note added: "12V 2A"
- note added: "40K intern pull up"
- note added: "ACTIONNEURS & SENSORS"
- note added: "BOOT & RST"
- note added: "Boot / DFU"
- note added: "COURANT"
- note added: "Classic mode"
- note added: "Cload = 2* (Ccrystal-Cstray)"
- note added: "Connection H30 -> OUT"
- note added: "Connectique OUT"
- note added: "Connector"
- note added: "Cristal"
- note added: "ESD"
- note added: "Electrovanne"
- note added: "FLASH Memory"
- note added: "Faire passer les pistes en dessous"
- note added: "Feed ressitor ~50R AN2867"
- note added: "LCSC bobine ?"
- note added: "LDO 3V3"
- note added: "MPX5010 ou MPRLS0025PA"
- note added: "Mounting Holes"
- note added: "NTC ? LM35 ?"
- note added: "POWER"
- note added: "PRESSION"
- note added: "RGB LED"
- note added: "Reverse polarity protection +Or gate (usb)"
- note added: "STM32 & CONN"
- note added: "STM32L4"
- note added: "Short cut protection"
- note added: "TEMPERATURE"
- note added: "USBC"
- note added: "VBUS = POWER if 12V off else VDiode <0"
- note added: "XL2EL89CLI-111YLC-16M"
- note added: "dimentionnement res / driver CC"
- note added: "only if DCDC can provide 95% of efficiency"
- note added: "only if ST reset during short cut"
- note added: "shield unconnected = easy soldering"
- note removed: "Connection H30 -> LIPO"
- note removed: "Connectique Lipo"
- note removed: "Electro vanne"
- note removed: "dimentionnement res"
- note removed: "evite le rebbot ?"
- note removed: "temperature pression ? Courant"
- moved on the sheet: C10, C11, C12, C5, C6, C7, C8, C9, D2, D3, D4, D8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

Commit message: Add files via upload
Parts:
- removed C11, C12: C_Polarized, symbol Device:C_Polarized
- removed C24: 220uF, symbol Device:C_Polarized
- removed J401: SWD, Connector_PinHeader_1.27mm:PinHeader_2x05_P1.27mm_Vertical_SMD, symbol Connector_Generic:Conn_02x05_Odd_Even
- removed Q4, Q8: PSMNR56-25YLEX, PSMNR56-25YLEX:PSMNR5830YLHX, symbol PSMNR56-25YLEX:PSMNR56-25YLEX
- removed R19: 0.1R, Resistor_SMD:R_0603_1608Metric, symbol Device:R
- removed R23, R24, R26: ?, Resistor_SMD:R_0603_1608Metric, symbol Device:R
- added C24, C26, C28: 470 uF, Capacitor_THT_Wurth_PT:CP_Wurth_WCAP-PTHT-P5D10L12.5, symbol Capacitor_Wurth_WCAP-PTHT:P5D10L12.5_870135375007
- added C29, C30, C31: 10 uF, Capacitor_SMD_Wurth:CP_Wurth_WCAP-ASLI-D4L5.5, symbol Capacitor_Wurth_WCAP-ASLI:D4L5.5_865080440002
- added C32: 2.2uF, Capacitor_SMD:C_0603_1608Metric, symbol Device:C
- added C33, C34: 100nF, Capacitor_SMD:C_0603_1608Metric, symbol Device:C
- added C35: C, Capacitor_SMD:C_0603_1608Metric, symbol Device:C
- added C36: 25 F, Capacitor_THT_Wurth:CP_Wurth_WCAP-STSC-P7.5D16L25, symbol Capacitor_Wurth_WCAP-STSC:P7.5D16L25_850617022001
- added C4: 220 uF, Capacitor_SMD_Wurth:CP_Wurth_WCAP-ASLI-D8L10.5, symbol Capacitor_Wurth_WCAP-ASLI:D8L10.5_865080453013
- added D13, D14, D15, D17, D18, D19, D20, D21, D22, D23, D24, D25: BAT54S-HF, BAT54S-HF:SOT95P240X115-3N, symbol BAT54S-HF:BAT54S-HF
- added IC4, IC5: ADS1115IDGSR, ADS1115IDGSR:SOP50P490X110-10N, symbol ADS1115IDGSR:ADS1115IDGSR
- added IC6: DRV8833CPWPR, DRV8833CPWPR:SOP65P640X120-17N, symbol DRV8833CPWPR:DRV8833CPWPR
- added IC7: LM358DR, LM358DR:SOIC127P600X175-8N, symbol LM358DR:LM358DR
- added J12: 62000411622, Connector_THT_Wurth:J_Wurth_WR-WTB_62000411622, symbol Connector_Wurth_WR-WTB:62000411622
- added J14, J15, J16: 62000211622, Connector_THT_Wurth:J_Wurth_WR-WTB_62000211622, symbol Connector_Wurth_WR-WTB:62000211622
- added J17, J18, J19, J20, J21, J22, J23, J24: 62000311622, Connector_THT_Wurth:J_Wurth_WR-WTB_62000311622, symbol Connector_Wurth_WR-WTB:62000311622
- added J2: SWD, Connector_PinHeader_1.27mm:PinHeader_2x07_P1.27mm_Vertical_SMD, symbol Connector_Generic_MountingPin:Conn_02x07_Odd_Even_MountingPin
- added JP3, JP4: ~, jumper_footprints:Jumper_3points_0402, symbol My_Jumper:jumper_3_points
- added R1, R55, R56, R62: 10K, Resistor_SMD:R_0603_1608Metric, symbol Device:R_Small
- added R29: 10K, Resistor_SMD:R_0603_1608Metric, symbol Device:R
- added R43, R47, R60: 220R, Resistor_SMD:R_0603_1608Metric, symbol Device:R
- added R52, R53, R66, R67, R68, R69, R70, R71, R72, R73: 22, Resistor_SMD:R_0603_1608Metric, symbol Device:R_Small
- added R59: 15K, Resistor_SMD:R_0603_1608Metric, symbol Device:R
- added R61: 2k2, Resistor_SMD:R_0603_1608Metric, symbol Device:R
- added R63: 12K, Resistor_SMD:R_0603_1608Metric, symbol Device:R
- added R64, R65: ?, Resistor_SMD:R_0603_1608Metric, symbol Device:R_Small
- added TP2: NFAULT, TestPoint:TestPoint_Pad_D2.0mm, symbol Connector:TestPoint
- added U3: LTC1044, LTC1044:SOIC127P600X175-8N, symbol Regulator_SwitchedCapacitor:LTC1044
- NT1: footprint (none) -> NetTie:NetTie-2_SMD_Pad2.0mm
- SW1: renamed from SW2; footprint 450404015514:450404015514 -> Button_Switch_SMD:Nidec_Copal_CAS-120A
- SW3: renamed from SW1; footprint 450404015514:450404015514 -> Button_Switch_SMD:Nidec_Copal_CAS-120A
- renumbered C21 to C1, C6 to C10, C17 to C11, C18 to C12, C7 to C13, C19 to C14, C8 to C15, C20 to C16, C9 to C17, C10 to C18, C65 to C19, C23 to C2, C1 to C20, C2 to C21, C212 to C22, C213 to C23, C3 to C25, C4 to C27, C22 to C3, C13 to C5, C5 to C6, C14 to C7, C15 to C8, C16 to C9, D10 to D1, D6 to D10, D7 to D11, D8 to D16, D9 to D2, D1 to D3, D3 to D4, D4 to D5, D2 to D6, D5 to D7, D201 to D8, D11 to D9, FB200 to FB1, J12 to J1, J7 to J11, J2 to J13, J4 to J3, J1 to J4, J3 to J5, J9 to J6, J5 to J7, J6 to J9, Q11 to Q10, Q13 to Q11, Q14 to Q2, Q2 to Q3, Q3 to Q4, Q10 to Q8, R3 to R10, R7 to R11, R8 to R12, R9 to R13, R30 to R14, R31 to R15, R10 to R16, R11 to R17, R12 to R18, R206 to R19, R32 to R2, R207 to R20, R208 to R21, R13 to R22, R35 to R23, R33 to R24, R14 to R25, R15 to R26, R16 to R27, R17 to R28, R29 to R3, R18 to R30, R43 to R31, R44 to R32, R20 to R33, R36 to R35, R39 to R36, R40 to R37, R21 to R38, R400 to R39, R28 to R4, R403 to R40, R401 to R41, R22 to R42, R402 to R44, R37 to R48, R38 to R49, R4 to R5, R41 to R50, R42 to R51, R48 to R54, R25 to R57, R27 to R58, R5 to R6, R6 to R7, R1 to R8, R2 to R9, SW4 to SW2, U9 to U2
Connections:
- net +12V: now also C31.1, IC6.12 (VM), IC7.8 (V+), U3.8 (V+)
- net +3V3: now also D13.2 (K), D14.2 (K), D15.2 (K), D17.2 (K), D18.2 (K), D19.2 (K), D20.2 (K), D21.2 (K), D22.2 (K), D23.2 (K), D24.2 (K), D25.2 (K), J12.4, J17.3, J18.3, J19.3, J2.3 (Pin_3), J20.3, J21.3, J22.3, J23.3, J24.3, JP3.2, JP4.2, R1.2, R55.1, R56.1, R62.1
- net +5V: now also C33.1, C34.1, IC4.8 (VDD), IC5.1 (ADDR), IC5.8 (VDD), JP3.1, JP4.1; no longer J10.2, J6.2
- net -H30: now also C31.2, C32.2, C4.2, IC6.13 (GND_1), IC6.17 (GND_2), R64.2, R65.2
- net -ST: now also C30.1, C33.2, C34.2, D13.1 (A), D14.1 (A), D15.1 (A), D17.1 (A), D18.1 (A), D19.1 (A), D20.1 (A), D21.1 (A), D22.1 (A), D23.1 (A), D24.1 (A), D25.1 (A), IC4.1 (ADDR), IC4.3 (GND), IC5.3 (GND), IC7.3 (IN1+), IC7.5 (IN2+), J12.1, J14.1, J17.1, J18.1, J19.1, J2.11 (Pin_11), J2.5 (Pin_5), J2.7 (Pin_7), J20.1, J21.1, J23.1, J24.1, U3.3 (GND)
- net ADC1_IN1+: now also D13.3 (K/A)
- net ADC1_IN2-: now also D20.3 (K/A)
- net ADC3_IN3+: now also D17.3 (K/A)
- net I2C1_SCA: now also IC4.9 (SDA), IC5.9 (SDA)
- net I2C1_SCL: now also IC4.10 (SCL), IC5.10 (SCL)
- net NRST: now also R1.1
- net OUT+: now also C24.1, C26.1, C28.1
- net OUT-: now also Q10.1 (S), Q10.2 (S), Q10.3 (S)
- net capa_out: now also C24.2, C26.2, C28.2, R29.1, R43.1, R47.1
- net at R40.2: now also J2.12 (Pin_12)
- net at R39.2: now also J2.4 (Pin_4)
- net at R41.2: now also J2.6 (Pin_6)
- net at R44.2: now also J2.8 (Pin_8)
- net at D11.2 (A): now also R29.2
- net at C6.1, D2.1 (K), IC1.2 (VIN)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: now also C4.1
- net BIN1: now reaches U1.35 (PB14)
- net BIN1: now also IC6.9 (BIN1)
- net BIN2: now reaches U1.36 (PB15)
- net BIN2: now also IC6.10 (BIN2)
- net AIN1: now reaches U1.38 (PC7)
- net AIN1: now also IC6.15 (AIN2)
- net AIN2: now reaches U1.40 (PC9)
- net AIN2: now also IC6.16 (AIN1)
- net UART5_TX: now reaches U1.53 (PC12)
- net UART5_TX: now also R53.2
- net UART5_RX: now reaches U1.54 (PD2)
- net UART5_RX: now also R52.2
- net ALERT1: now reaches U1.61 (PB8)
- net ALERT1: now also IC4.2 (ALERT/RDY), R55.2
- net ALERT2: now reaches U1.62 (PB9)
- net ALERT2: now also IC5.2 (ALERT/RDY), R56.2
- net ADC3_IN4- renamed ADC2_IN4
- net ADC2_IN4: now also D23.3 (K/A), IC7.7 (OUT2), R61.2
- net Capa_out: no longer names the net of Q10.5 (D)
- net Capa_out: now also R43.2, R47.2
- new net: C35.1, IC7.2 (IN1-), J14.2, R60.1
- new net: C35.2, IC7.1 (OUT1), R60.2, R63.2
- new net: IC7.6 (IN2-), R59.2, R61.1, R63.1
- new net: J12.2, R53.1
- new net: J23.2, R72.1
- new net: J19.2, R68.1
- new net: J10.2, JP4.3
- new net: J17.2, R66.1
- new net: J20.2, R69.1
- new net: IC6.4 (AOUT2), J15.1
- new net: IC6.2 (AOUT1), J15.2
- new net: C29.1, U3.2 (CAP+)
- new net: C29.2, U3.4 (CAP-)
- new net: J22.2, R71.1
- new net: J12.3, R52.1
- new net: IC6.5 (BOUT2), J16.1
- new net: IC6.7 (BOUT1), J16.2
- new net: J6.2, JP3.3
- new net: J18.2, R67.1
- new net: J24.2, R73.1
- new net: J21.2, R70.1
- new net -12V: C30.2, IC7.4 (V-), R59.1, U3.5 (VOUT)
- new net ADC1_EX0: D14.3 (K/A), IC4.4 (AIN0), R66.2
- new net ADC1_EX1: D18.3 (K/A), IC4.5 (AIN1), R67.2
- new net ADC1_EX2: D21.3 (K/A), IC4.6 (AIN2), R68.2
- new net ADC1_EX3: D24.3 (K/A), IC4.7 (AIN3), R69.2
- new net ADC2_EX0: D15.3 (K/A), IC5.4 (AIN0), R70.2
- new net ADC2_EX1: D19.3 (K/A), IC5.5 (AIN1), R71.2
- new net ADC2_EX2: D22.3 (K/A), IC5.6 (AIN2), R72.2
- new net ADC2_EX3: D25.3 (K/A), IC5.7 (AIN3), R73.2
- new net AISEN: IC6.3 (AISEN), R64.1
- new net BISEN: IC6.6 (BISEN), R65.1
- new net NFAULT: IC6.1 (NSLEEP), IC6.8 (NFAULT), R62.2, TP2.1
- new net VINT: C32.1
- no-connect marks 9 -> 26
Other:
- note added: "(+-30mA -> 0-2.3V)"
- note added: "14 pin (match avec ST-Link)"
- note added: "ADC Security"
- note added: "ADC's ST"
- note added: "Ajout led cf note iphone"
- note added: "BQ33100PW"
- note added: "EXTERNAL ADC & PROTECTIONS"
- note added: "EXTI"
- note added: "External ADC"
- note added: "FAN"
- note added: "FAN driver"
- note added: "I2C"
- note added: "ID 0x48"
- note added: "ID 0x49"
- note added: "Inverseur de tension"
- note added: "Isens (optionnal)"
- note added: "LCSC ref : XL2EL89CLI-111YLC-16M"
- note added: "LM35"
- note added: "LTC3350EUHF#TRPBF"
- note added: "Load swicth TSP22981 impossible car up side"
- note added: "MPRLS0025PA"
- note added: "MPX5010"
- note added: "Main H30 Circuit"
- note added: "Moteur tire sur les super capa en serie (20F 12V) hydrogene charge constament les capa (diode antiretour ideal ?)"
- note added: "NTC sondes"
- note added: "OUTPUT"
- note added: "PRESSION & TEMPERATURE"
- note added: "PT100"
- note added: "PWR"
- note added: "SDA 0x4A SCL 0x4B"
- note added: "SWD & SPI"
- note added: "UART"
- note added: "capteur courant divise par 1000. Donc : 30A = 30mA a lire"
- note added: "esr 25mR"
- note removed: "LCSC bobine ?"
- note removed: "MPX5010 ou MPRLS0025PA"
- note removed: "NTC ? LM35 ?"
- note removed: "PRESSION"
- note removed: "Super capa"
- note removed: "TEMPERATURE"
- note removed: "XL2EL89CLI-111YLC-16M"
- note removed: "dimentionnement res / driver CC"
- note removed: "dimnetionner reistance de decharge"
- note removed: "mettre des capas (100nf et decoupling?)"
- note removed: "pin stable avant boot"
- moved on the sheet: C10, C13, C15, C17, C18, C19, C2, C20, C21, C22, C23, C25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

Commit message: upload V1
Parts:
- removed C4: 220 uF, Capacitor_SMD_Wurth:CP_Wurth_WCAP-ASLI-D8L10.5, symbol Capacitor_Wurth_WCAP-ASLI:D8L10.5_865080453013
- added C25: 100nF, Capacitor_SMD:C_0603_1608Metric, symbol Device:C
- added C29, C31, C32: 470 uF, Capacitor_THT_Wurth_PT:CP_Wurth_WCAP-PTHT-P5D10L12.5, symbol Capacitor_Wurth_WCAP-PTHT:P5D10L12.5_870135375007
- added C4: 47 uF, Capacitor_SMD_Wurth:CP_Wurth_WCAP-ASLI-D6.3L5.5, symbol Capacitor_Wurth_WCAP-ASLI:D6.3L5.5_S8650804430071
- added D13, D3: RED, LED_SMD:LED_0603_1608Metric, symbol Device:LED
- added Q11, Q4: 2N7002, Package_TO_SOT_SMD:SOT-23, symbol Transistor_FET:2N7002
- added R10, R51: 2.2K, Resistor_SMD:R_0603_1608Metric, symbol Device:R_Small
- added R50, R9: 220, Resistor_SMD:R_0603_1608Metric, symbol Device:R_Small
- added R8: 220R, Resistor_SMD:R_0603_1608Metric, symbol Device:R
- added TP2: Gate_H30->OUT, TestPoint:TestPoint_Pad_D2.0mm, symbol Connector:TestPoint
- renumbered C25 to C26, C26 to C27, C27 to C28, C28 to C30, C29 to C33, C30 to C34, C31 to C35, C32 to C36, C33 to C37, C34 to C38, C35 to C39, C36 to C40, D9 to D10, D10 to D11, D11 to D12, D12 to D14, D13 to D15, D14 to D16, D15 to D17, D16 to D18, D17 to D19, D18 to D20, D19 to D21, D20 to D22, D21 to D23, D22 to D24, D23 to D25, D24 to D26, D25 to D27, D3 to D4, D4 to D5, D5 to D6, D6 to D7, D7 to D8, D8 to D9, Q9 to Q10, Q10 to Q12, Q11 to Q13, Q12 to Q14, Q4 to Q5, Q5 to Q6, Q6 to Q7, Q7 to Q8, Q8 to Q9, R8 to R11, R9 to R12, R10 to R13, R11 to R14, R12 to R15, R13 to R16, R14 to R17, R15 to R18, R16 to R19, R17 to R20, R18 to R21, R19 to R22, R20 to R23, R21 to R24, R22 to R25, R23 to R26, R24 to R27, R25 to R28, R26 to R29, R27 to R30, R28 to R31, R30 to R32, R29 to R33, R33 to R34, R31 to R35, R32 to R36, R34 to R37, R35 to R38, R36 to R39, R37 to R40, R38 to R41, R39 to R42, R40 to R43, R41 to R44, R42 to R45, R44 to R46, R45 to R47, R46 to R48, R43 to R49, R47 to R52, R48 to R53, R49 to R54, R50 to R55, R51 to R56, R52 to R57, R53 to R58, R54 to R59, R55 to R60, R56 to R61, R57 to R62, R58 to R63, R59 to R64, R60 to R65, R61 to R66, R62 to R67, R63 to R68, R64 to R69, R65 to R70, R66 to R71, R67 to R72, R68 to R73, R69 to R74, R70 to R75, R71 to R76, R72 to R77, R73 to R78, TP2 to TP3
Connections:
- net +3V3: now also R10.1, R51.1
- net -H30: now also C4.2, Q11.2 (S), Q4.2 (S)
- net Gate_H30-OUT-: now also TP2.1
- net OUT+: now also C29.1, C31.1, C32.1
- net OUT-: now also C25.2
- net capa_out: now also Q12.5 (D), R49.2, R52.2; no longer C24.2, C27.2, C30.2, Q10.5 (D), R49.1, R52.1
- net at C6.1, D2.1 (K), IC1.2 (VIN)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: now also C4.1
- net LED_Capa: now reaches Q9.3 (D), R41.2, R45.1
- net LED_Capa: now also R50.1
- net at Q10.4 (G), R32.1, R34.1: now also C25.1
- net LED_Short: now reaches Q3.2 (S), R7.2
- net LED_Short: now also R8.1, R9.1; no longer Q5.4 (G)
- new net: Q4.1 (G), R9.2
- new net: D3.1 (K), Q4.3 (D)
- new net: D3.2 (A), R10.2
- new net: C24.2, C27.2, C29.2, C30.2, C31.2, C32.2, Q10.5 (D), R49.1, R52.1
- new net: D13.1 (K), Q11.3 (D)
- new net: D13.2 (A), R51.2
- new net: Q5.4 (G), R8.2
- new net: Q11.1 (G), R50.2
Other:
- note added: "Res decharge"
- note added: "Soft start Vg(t)=Vin*(1−e^(−t/(R×C)))"
- note added: "Tuner l eprinte pluseir trou pour capa biface + petit capa"
- note removed: "Ajout led cf note iphone"
- moved on the sheet: C24, C30, Q12, Q5, R32, R34, R49, R52, R7

Commit message: V1
Parts:
- removed C40: 25 F, Capacitor_THT_Wurth:CP_Wurth_WCAP-STSC-P7.5D16L25, symbol Capacitor_Wurth_WCAP-STSC:P7.5D16L25_850617022001
- added D1: RED, LED_SMD:LED_0603_1608Metric, symbol Device:LED
- added R2: 5K1, Resistor_SMD:R_0603_1608Metric, symbol Device:R_Small
- added TP1: SDA, TestPoint:TestPoint_Pad_D1.5mm, symbol Connector:TestPoint
- added TP2: SCL, TestPoint:TestPoint_Pad_D1.5mm, symbol Connector:TestPoint
- added TP3: LTC gate, TestPoint:TestPoint_Pad_D1.5mm, symbol Connector:TestPoint
- added TP6: V_Reverse, TestPoint:TestPoint_Pad_D1.5mm, symbol Connector:TestPoint
- C4: now not fitted
- H3: value MountingHole_Pad -> Pad 3.2 mm M3
- R70: renamed from R69; value ? -> 0R; now fitted
- R79: renamed from R70; value ? -> 0R; now fitted
- TP4: renamed from TP1; footprint TestPoint:TestPoint_Pad_D2.0mm -> TestPoint:TestPoint_Pad_D1.5mm
- TP5: renamed from TP2; footprint TestPoint:TestPoint_Pad_D2.0mm -> TestPoint:TestPoint_Pad_D1.5mm
- TP7: renamed from TP3; footprint TestPoint:TestPoint_Pad_D2.0mm -> TestPoint:TestPoint_Pad_D1.5mm
- renumbered D9 to D10, D10 to D11, D11 to D12, D12 to D13, D13 to D14, D14 to D15, D15 to D16, D16 to D17, D17 to D18, D18 to D19, D1 to D2, D19 to D20, D20 to D21, D21 to D22, D22 to D23, D23 to D24, D24 to D25, D25 to D26, D26 to D27, D27 to D28, D2 to D3, D3 to D4, D4 to D5, D5 to D6, D6 to D7, D7 to D8, D8 to D9, R9 to R10, R10 to R11, R11 to R12, R12 to R13, R13 to R14, R14 to R15, R15 to R16, R16 to R17, R17 to R18, R18 to R19, R19 to R20, R20 to R21, R21 to R22, R22 to R23, R23 to R24, R24 to R25, R25 to R26, R26 to R27, R27 to R28, R28 to R29, R2 to R3, R29 to R30, R30 to R31, R31 to R32, R32 to R33, R33 to R34, R34 to R35, R35 to R36, R36 to R37, R37 to R38, R38 to R39, R3 to R4, R39 to R40, R40 to R41, R41 to R42, R42 to R43, R43 to R44, R44 to R45, R45 to R46, R46 to R47, R47 to R48, R48 to R49, R4 to R5, R49 to R50, R50 to R51, R51 to R52, R52 to R53, R53 to R54, R54 to R55, R55 to R56, R56 to R57, R57 to R58, R58 to R59, R5 to R6, R59 to R60, R60 to R61, R61 to R62, R62 to R63, R63 to R64, R64 to R65, R65 to R66, R66 to R67, R67 to R68, R68 to R69, R6 to R7, R7 to R8, R8 to R9
Connections:
- net GND is gone; now on net -ST: R27.1, R28.1
- net +12V: now also R2.1
- net -12V: now also TP6.1
- net -ST: now also J22.1
- net I2C1_SCL: now also TP2.1
- net LTC gate: now also TP3.1
- net VINT: now also IC6.14 (VINT)
- net at F1.2, Q2.3 (D): now also D1.1 (K)
- net I2C1_SCA renamed I2C1_SDA
- net I2C1_SDA: now also TP1.1
- new net: D1.2 (A), R2.2
- no-connect marks 26 -> 27
Other:
- note added: "Isens (optionnal) shunt"
- note added: "RUN"
- note added: "To DCDC via Diode"
- note removed: "BQ33100PW"
- note removed: "Classic mode"
- note removed: "Isens (optionnal)"
- note removed: "LTC3350EUHF#TRPBF"
- note removed: "Moteur tire sur les super capa en serie (20F 12V) hydrogene charge constament les capa (diode antiretour ideal ?)"
- note removed: "VBUS = POWER if 12V off else VDiode <0"
- note removed: "esr 25mR"
- moved on the sheet: C22, C35, R18, R19, SW1

Commit message: Add files via upload
Parts:
- removed J10, J13, J14, J15, J16, J6: 62000211622, Connector_THT_Wurth:J_Wurth_WR-WTB_62000211622, symbol Connector_Wurth_WR-WTB:62000211622
- removed J11: 62000611622, Connector_THT_Wurth:J_Wurth_WR-WTB_62000611622, symbol Connector_Wurth_WR-WTB:62000611622
- removed J12, J3, J4, J5, J7, J8, J9: 62000411622, Connector_THT_Wurth:J_Wurth_WR-WTB_62000411622, symbol Connector_Wurth_WR-WTB:62000411622
- removed J17, J18, J19, J20, J21, J22, J23, J24: 62000311622, Connector_THT_Wurth:J_Wurth_WR-WTB_62000311622, symbol Connector_Wurth_WR-WTB:62000311622
- added J10, J11, J13, J4, J5, J6, J9: 653004114822, Connector_THT_Wurth:J_Wurth_WR-WTB_653004114822, symbol Connector_Wurth_WR-WTB:653004114822
- added J12, J16, J17, J18, J19, J7: 653002114822, Connector_THT_Wurth:J_Wurth_WR-WTB_653002114822, symbol Connector_Wurth_WR-WTB:653002114822
- added J14: 653006114822, Connector_THT_Wurth:J_Wurth_WR-WTB_653006114822, symbol Connector_Wurth_WR-WTB:653006114822
- added J20, J21, J22, J23, J24, J25, J26, J27: 653003114822, Connector_THT_Wurth:J_Wurth_WR-WTB_653003114822, symbol Connector_Wurth_WR-WTB:653003114822
- added J8: TC2030, Connector:Tag-Connect_TC2030-IDC-NL_2x03_P1.27mm_Vertical, symbol Connector:TC2030
- added LS1: CMT-8530S-SMT-TR, CMT-8530S-SMT-TR:CMT8530SSMTTR, symbol CMT-8530S-SMT-TR:CMT-8530S-SMT-TR
- added Q8: 2N7002, Package_TO_SOT_SMD:SOT-23, symbol Transistor_FET:2N7002
- added R31: 0, Resistor_SMD:R_0603_1608Metric, symbol Device:R_Small
- added R32: 220, Resistor_SMD:R_0603_1608Metric, symbol Device:R_Small
- added TP6: V_Reverse, TestPoint:TestPoint_Pad_D1.5mm, symbol Connector:TestPoint
- renumbered C23 to C22, C22 to C23, Q1 to J1, Q13 to J15, J1 to J2, J2 to J3, Q2 to Q1, Q14 to Q13, Q3 to Q2, Q4 to Q3, Q5 to Q4, Q6 to Q5, Q7 to Q6, Q8 to Q7, R31 to R33, R32 to R34, R33 to R35, R34 to R36, R35 to R37, R36 to R38, R37 to R39, R43 to R40, R45 to R41, R47 to R42, R44 to R43, R38 to R44, R39 to R45, R40 to R46, R41 to R47, R42 to R48, R46 to R49, R48 to R50, R49 to R51, R50 to R52, R51 to R53, R52 to R54, R53 to R55, R54 to R56, R55 to R57, R56 to R58, R57 to R59, R58 to R60, R59 to R61, R60 to R62, R61 to R63, R62 to R64, R63 to R65, R64 to R66, R65 to R67, R66 to R68, R67 to R69, R68 to R70, R69 to R71, R70 to R72, R71 to R73, R72 to R74, R73 to R75, R74 to R76, R75 to R77, R76 to R78, R77 to R79, R78 to R80, R79 to R81, TP6 to TP7, TP7 to TP8
Connections:
- net +3V3: now also J10.4, J11.4, J13.4, J14.6, J20.3, J21.3, J22.3, J23.3, J24.3, J25.3, J26.3, J27.3, J4.4, J5.4, J6.4, J8.1, J9.4, LS1.1 (+)
- net -H30: now also J16.1
- net -ST: now also J10.1, J11.1, J12.1, J13.1, J14.1, J17.1, J20.1, J21.1, J22.1, J23.1, J24.1, J25.1, J26.1, J27.1, J4.1, J5.1, J6.1, J7.1, J8.5, J9.1, Q8.2 (S), TP6.1
- net NRST: now also J8.3
- net SPI1_CS: now also J14.5
- net SPI1_MISO: now also J14.3
- net SPI1_MOSI: now also J14.4
- net SPI1_SCK: now also J14.2
- net SWCLK: now also J8.4
- net SWDIO: now also J8.2
- net SWO: now also J8.6
- net at R47.1: now also J6.2
- net at R46.1: now also J6.3
- net at C39.1, IC7.2 (IN1-), R68.1: now also J17.2
- net at R57.1: now also J10.2
- net TIM1_CH3: now reaches U1.43 (PA10)
- net TIM1_CH3: now also R32.1
- net at R61.1: now also J13.2
- net at R51.1: now also J9.2
- net at R50.1: now also J9.3
- net at R79.1: now also J26.2
- net at R75.1: now also J22.2
- net at JP4.3: now also J12.2
- net at R59.1: now also J11.2
- net at R73.1: now also J20.2
- net at R76.1: now also J23.2
- net at IC6.4 (AOUT2): now also J18.1
- net at IC6.2 (AOUT1): now also J18.2
- net at R45.1: now also J5.2
- net at R44.1: now also J5.3
- net at R58.1: now also J11.3
- net at R78.1: now also J25.2
- net at R56.1: now also J10.3
- net at R60.1: now also J13.3
- net at IC6.5 (BOUT2): now also J19.2
- net at IC6.7 (BOUT1): now also J19.1
- net at JP3.3: now also J7.2
- net at R74.1: now also J21.2
- net at R38.1: now also J4.3
- net at R80.1: now also J27.2
- net at R39.1: now also J4.2
- net at D19.1 (K), Q13.3 (D): now also J16.2
- net at R77.1: now also J24.2
- new net: Q8.1 (G), R32.2
- new net: Q8.3 (D), R31.1
- new net: LS1.2 (-), R31.2
- no-connect marks 27 -> 28
Other:
- note added: "Buzzer"
- note added: "Code borg : 1423"
- note added: "REF"
- note added: "Tag Connect"
- note removed: "PRESSION & TEMPERATURE"
- moved on the sheet: J3, R40, R41, R42, R43, R69
