File: PCB/H30_controler_board.kicad_sch (KiCad schematic)
At the start: 224 parts, among them IC1 MP2338GTL-P, IC2 LTC4359IMS8#PBF, IC3 W25N01GVZEIG, IC4 ADS1115IDGSR, IC5 ADS1115IDGSR, IC6 DRV8833CPWPR, IC7 LM358DR, J1 XT60_YELLOW, J10 653004114822, J11 653004114822, J12 653002114822, J13 653004114822, J14 653006114822, J15 XT60_YELLOW, J16 653002114822, J17 653002114822, J18 653002114822, J19 653002114822, J2 USB_C_Receptacle_USB2.0_14P, J20 653003114822, J21 653003114822, J22 653003114822, J23 653003114822, J24 653003114822, J25 653003114822, J26 653003114822, J27 653003114822, J3 SWD, J4 653004114822, J5 653004114822, J6 653004114822, J7 653002114822, J8 TC2030, J9 653004114822, Q1 AO3401A, Q10 PSMNR56-25YLEX, Q11 2N7002, Q12 PSMNR56-25YLEX, Q13 SI2301-TP, Q2 SI2301-TP, Q3 2N7002, Q4 PSMNR56-25YLEX, Q5 PSMNR56-25YLEX, Q6 SI2301-TP, Q7 PSMNR56-25YLEX, Q8 2N7002, Q9 SI2301-TP, SW1 SW_Nidec_CAS-120A1, SW3 SW_Nidec_CAS-120A1, U1 STM32L476RCTx, U2 USBLC6-2SC6, U3 LTC1044, Y1 16MHz

Commit message: V1.1
Parts:
- removed C12: 100nf, Capacitor_SMD:C_0603_1608Metric, symbol Device:C_Small
- removed C31: 470 uF, Capacitor_THT_Wurth_PT:CP_Wurth_WCAP-PTHT-P5D10L12.5, symbol Capacitor_Wurth_WCAP-PTHT:P5D10L12.5_870135375007
- removed C35: 10 uF, Capacitor_SMD_Wurth:CP_Wurth_WCAP-ASLI-D4L5.5, symbol Capacitor_Wurth_WCAP-ASLI:D4L5.5_865080440002
- removed D12: STPS2L30A, STPS2L30A:DIOM5126X265N, symbol STPS2L30A:STPS2L30A
- removed J1: XT60_YELLOW, XT60:AMASS_XT60PB-M, symbol XT60_YELLOW:XT60_YELLOW
- removed J11: 653004114822, Connector_THT_Wurth:J_Wurth_WR-WTB_653004114822, symbol Connector_Wurth_WR-WTB:653004114822
- removed R33: 10K, Resistor_SMD:R_0603_1608Metric, symbol Device:R
- added C12: 10uF, Capacitor_SMD:C_1210_3225Metric, symbol Device:C
- added J1: 662102145021, MPC3_Wurth:J_Wurth_WR-MPC3_662102145021, symbol Connector_Wurth_WR-MPC3:662102145021
- added J11, J28: 653006114822, Connector_THT_Wurth:J_Wurth_WR-WTB_653006114822, symbol Connector_Wurth_WR-WTB:653006114822
- added J29: Conn_02x07_Odd_Even, Connector_PinSocket_1.27mm:PinSocket_2x07_P1.27mm_Vertical, symbol Connector_Generic:Conn_02x07_Odd_Even
- added J30: Conn_01x14_Socket, Connector_PinSocket_2.54mm:PinSocket_2x07_P2.54mm_Vertical, symbol Connector:Conn_01x14_Socket
- J13: now left out of the parts list
- J18, J19: value 653002114822 -> 653102131822; footprint Connector_THT_Wurth:J_Wurth_WR-WTB_653002114822 -> Connector_SMD_Wurth:J_Wurth_WR-WTB_653102131822
- J3: footprint Connector_PinHeader_1.27mm:PinHeader_2x07_P1.27mm_Vertical_SMD -> Connector_PinHeader_1.27mm:PinHeader_2x07_P1.27mm_Vertical
- R1, R38, R39, R40, R41, R42, R43, R44, R45, R46, R47, R50, R51, R56, R57, R58, R59, R73, R74, R75, R76, R77, R78, R79, R80: footprint Resistor_SMD:R_0603_1608Metric -> Resistor_SMD:R_0402_1005Metric
- R52, R55: footprint Resistor_SMD:R_0603_1608Metric -> Resistor_SMD:R_1210_3225Metric
- R60, R61: footprint Resistor_SMD:R_0603_1608Metric -> Resistor_SMD:R_0402_1005Metric; now left out of the parts list
- SW1, SW3: footprint Button_Switch_SMD:Nidec_Copal_CAS-120A -> 450404015514:450404015514
Connections:
- net +12V: no longer IC6.12 (VM)
- net +3V3: now also C37.1, C38.1, IC4.8 (VDD), IC5.1 (ADDR), IC5.8 (VDD), JP3.3, JP4.3, J11.6, J28.6; no longer JP3.2, JP4.2, R54.1
- net +5V: no longer C37.1, C38.1, IC4.8 (VDD), IC5.1 (ADDR), IC5.8 (VDD)
- net +H30: now also IC6.12 (VM), C12.1, J1.2
- net -H30: now also C12.2, J1.1; no longer C10.2, C15.2, C17.2, C4.2, C6.2, D9.1 (K), H1.1, H2.1, H3.1, H4.1, IC1.4 (GND), Q1.1 (G), R14.1, R17.1
- net -ST: now also C10.2, C15.2, C17.2, C4.2, C6.2, D9.1 (K), IC1.4 (GND), Q1.1 (G), R14.1, R17.1, J11.1, J28.1
- net ALERT1: now also J11.3, J28.3
- net ALERT2: now also J11.2, J28.2
- net I2C1_SCL: now also J28.4
- net I2C1_SDA: now also J28.5
- net OUT+: now also R36.1, R52.1, R54.1, R55.1
- net OUT-: no longer Q12.1 (S), Q12.2 (S), Q12.3 (S)
- net capa_out: now also C24.2, C27.2, C29.2, C30.2, C32.2, Q10.5 (D), Q12.1 (S), Q12.2 (S), Q12.3 (S); no longer Q12.5 (D), R36.1, R52.2, R55.2
- net at R59.1: now also J11.4
- net at R58.1: now also J11.5
- net at J12.2: now also JP4.2; no longer JP4.3
- net at J19.1: now also IC6.5 (BOUT2); no longer IC6.7 (BOUT1)
- net at J19.2: now also IC6.7 (BOUT1); no longer IC6.5 (BOUT2)
- net at J7.2: now also JP3.2; no longer JP3.3
- new net: Q12.5 (D), R52.2, R55.2
- new net 1: J29.1 (Pin_1), J30.1 (Pin_1)
- new net 10: J29.10 (Pin_10), J30.10 (Pin_10)
- new net 11: J29.11 (Pin_11), J30.11 (Pin_11)
- new net 12: J29.12 (Pin_12), J30.12 (Pin_12)
- new net 13: J29.13 (Pin_13), J30.13 (Pin_13)
- new net 14: J29.14 (Pin_14), J30.14 (Pin_14)
- new net 2: J29.2 (Pin_2), J30.2 (Pin_2)
- new net 3: J29.3 (Pin_3), J30.3 (Pin_3)
- new net 4: J29.4 (Pin_4), J30.4 (Pin_4)
- new net 5: J29.5 (Pin_5), J30.5 (Pin_5)
- new net 6: J29.6 (Pin_6), J30.6 (Pin_6)
- new net 7: J29.7 (Pin_7), J30.7 (Pin_7)
- new net 8: J29.8 (Pin_8), J30.8 (Pin_8)
- new net 9: J29.9 (Pin_9), J30.9 (Pin_9)
Other:
- note added: "-ST ? DCDC ?"
- note added: "I2C & SPI"
- note added: "Res decharge 1210"
- note added: "SWD"
- note added: "~5A max"
- note removed: "I2C"
- note removed: "Male = no power provider Female = power provider here XT60 Male"
- note removed: "Res decharge"
- note removed: "SWD & SPI"
- moved on the sheet: C32, C37, C38, D13, D14, J14, J6, Q11, Q12, R36, R46, R47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

Commit message: PCB V1.1
Parts:
- C8: footprint Capacitor_SMD:C_0603_1608Metric -> Capacitor_SMD:C_0402_1005Metric
Other:
- company: H2 ECE Team -> H2GP ECE Team
Changed lines of the file:
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@@
 		(title "Manager for H30 hydrogene stack")
 		(date "2026-04-28")
-		(rev "1.0")
-		(company "H2 ECE Team")
+		(rev "1.1")
+		(company "H2GP ECE Team")
 		(comment 1 "Maxence HEROUX")
 	)
@@
 			)
 		)
-		(property "Footprint" "Capacitor_SMD:C_0603_1608Metric"
+		(property "Footprint" "Capacitor_SMD:C_0402_1005Metric"
 			(at 113.03 265.43 0)
 			(effects
