File: PCB/H30_controler_board.kicad_sch (KiCad schematic)
At the start: 223 parts, among them IC1 MP2338GTL-P, IC2 LTC4359IMS8#PBF, IC3 W25N01GVZEIG, IC4 ADS1115IDGSR, IC5 ADS1115IDGSR, IC6 DRV8833CPWPR, IC7 LM358DR, J1 662102145021, J10 653004114822, J11 653006114822, J12 653002114822, J13 653004114822, J14 653006114822, J15 XT60_YELLOW, J16 653002114822, J17 653002114822, J18 653102131822, J19 653102131822, J2 USB_C_Receptacle_USB2.0_14P, J20 653003114822, J21 653003114822, J22 653003114822, J23 653003114822, J24 653003114822, J25 653003114822, J26 653003114822, J27 653003114822, J28 653006114822, J29 Conn_02x07_Odd_Even, J3 SWD, J30 Conn_01x14_Socket, J4 653004114822, J5 653004114822, J6 653004114822, J7 653002114822, J8 TC2030, J9 653004114822, Q1 AO3401A, Q10 PSMNR56-25YLEX, Q11 2N7002, Q12 PSMNR56-25YLEX, Q13 SI2301-TP, Q2 SI2301-TP, Q3 2N7002, Q4 PSMNR56-25YLEX, Q5 PSMNR56-25YLEX, Q6 SI2301-TP, Q7 PSMNR56-25YLEX, Q8 2N7002, Q9 SI2301-TP, SW1 SW_Nidec_CAS-120A1, SW3 SW_Nidec_CAS-120A1, U1 STM32L476RCTx, U2 USBLC6-2SC6, U3 LTC1044, Y1 16MHz

Commit message: V1.2
Parts:
- removed C33, C34: 10 uF, Capacitor_SMD_Wurth:CP_Wurth_WCAP-ASLI-D4L5.5, symbol Capacitor_Wurth_WCAP-ASLI:D4L5.5_865080440002
- removed C39: C, Capacitor_SMD:C_0603_1608Metric, symbol Device:C
- removed IC7: LM358DR, LM358DR:SOIC127P600X175-8N, symbol LM358DR:LM358DR
- removed J17: 653002114822, Connector_THT_Wurth:J_Wurth_WR-WTB_653002114822, symbol Connector_Wurth_WR-WTB:653002114822
- removed R67: 15K, Resistor_SMD:R_0603_1608Metric, symbol Device:R
- removed R68: 220R, Resistor_SMD:R_0603_1608Metric, symbol Device:R
- removed R69: 2k2, Resistor_SMD:R_0603_1608Metric, symbol Device:R
- removed R71: 12K, Resistor_SMD:R_0603_1608Metric, symbol Device:R
- removed TP7: V_Reverse, TestPoint:TestPoint_Pad_D1.5mm, symbol Connector:TestPoint
- removed U3: LTC1044, LTC1044:SOIC127P600X175-8N, symbol Regulator_SwitchedCapacitor:LTC1044
- added IC8: 114993390, 114993390:114993390, symbol 114993390:114993390
- added JP5: ~, jumper_footprints:Jumper_3points_0402, symbol My_Jumper:jumper_3_points
Connections:
- net +3V3: now also IC8.8 (VCC), JP5.1
- net -ST: now also IC8.10 (GND_2), IC8.7 (GND_1), JP5.3
- net SPI1_MISO: now also IC8.2 (MISO)
- net SPI1_MOSI: now also IC8.3 (MOSI)
- net SPI1_SCK: now also IC8.4 (SCK)
- net SPI1_NSS: now reaches U1.20 (PA4)
- net SPI1_NSS: now also IC8.6 (NSS)
- net GPIO_BUSY: now reaches U1.28 (PB2)
- net GPIO_BUSY: now also IC8.11 (BUSY)
- net LORA_NRST: now reaches U1.33 (PB12)
- net LORA_NRST: now also IC8.5 (NRST)
- net GPIO_EXTI13: now reaches U1.34 (PB13)
- net GPIO_EXTI13: now also IC8.12 (DIO1)
- new net: IC8.1 (RF_SW_), JP5.2
- no-connect marks 28 -> 26
Other:
- note added: "ACTIONNEURS"
- note added: "LORA"
- note added: "LORA : WIO SX1262"
- note added: "NEW"
- note added: "RX"
- note added: "TX"
- note added: "Test point pour des tests devices"
- note removed: "(+-30mA -> 0-2.3V)"
- note removed: "ACTIONNEURS & SENSORS"
- note removed: "COURANT"
- note removed: "Inverseur de tension"
- note removed: "capteur courant divise par 1000. Donc : 30A = 30mA a lire"
- moved on the sheet: C20, C21, C26, C28, D11, D15, D19, D8, D9, J16, LS1, PS1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
