File: PCB/H30_controler_board.kicad_pcb (KiCad board)
At the start: 2 copper layers, 15 parts, among them IC1 LTC4359IMS8#PBF, Q1 PSMNR56-25YLEX, Q2 PSMNR56-25YLEX, Q3 PSMNR56-25YLEX, Q4 PSMNR56-25YLEX, Q5 PSMNR56-25YLEX, Q6 PSMNR56-25YLEX, Q8 SI2301-TP, Q9 SI2301-TP, U3 STM32L476RCTx

Commit message: Add files via upload
Parts:
- added C2: 22uF, Capacitor_SMD:C_0603_1608Metric, F.Cu at (88.3, 36.9)
- added C3: 22nF, Capacitor_SMD:C_0603_1608Metric, F.Cu at (88.3, 39.4)
- added C4: 22uF, Capacitor_SMD:C_0603_1608Metric, F.Cu at (88.3, 41.9)
- added C5: 22uF, Capacitor_SMD:C_0603_1608Metric, F.Cu at (88.3, 44.5)
- added C6: 0.1uF, Capacitor_SMD:C_0603_1608Metric, F.Cu at (88.3, 47.0)
- added D2: SS34, Diode_SMD:D_SMA, F.Cu at (110.9, 57.0)
- added D3: LED, LED_SMD:LED_0603_1608Metric, F.Cu at (92.9, 61.6)
- added D4: SMAT70A-13-F, SMAT70A-13-F:DIOM5226X230N, F.Cu at (102.8, 56.8)
- added D5: SMAJ24A, SMAJ24A:DIOM4325X250N, F.Cu at (102.9, 61.0)
- added IC2: MP2338GTL-P, MP2338GTL:SOTFL50P160X60-8N, F.Cu at (108.6, 61.1)
- added J1: Conn_01x02_Socket, Connector_PinSocket_2.54mm:PinSocket_1x02_P2.54mm_Vertical, F.Cu at (88.6, 58.1)
- added Q10: XT60_YELLOW, XT60:AMASS_XT60PB-M, F.Cu at (107.4, 40.4)
- added Q11: XT60_YELLOW, XT60:AMASS_XT60PB-F, F.Cu at (107.4, 50.0)
- added Q7: SI2301-TP, SI2301:SOT95P237X125-3N, F.Cu at (93.3, 58.0)
- added R10: 90.9K, Resistor_SMD:R_0603_1608Metric, F.Cu at (92.3, 44.5)
- added R11: 10K, Resistor_SMD:R_0603_1608Metric, F.Cu at (92.3, 47.0)
- added R12: 10K, Resistor_SMD:R_0603_1608Metric, F.Cu at (92.3, 49.5)
- added R13: 2.2K, Resistor_SMD:R_0603_1608Metric, F.Cu at (92.3, 52.0)
- added R14: 10K, Resistor_SMD:R_0603_1608Metric, F.Cu at (92.3, 54.5)
- added R15: ?, Resistor_SMD:R_0603_1608Metric, F.Cu at (96.3, 36.9)
- added R16: 10K, Resistor_SMD:R_0603_1608Metric, F.Cu at (96.3, 39.4)
- added R17: 2.2K, Resistor_SMD:R_0603_1608Metric, F.Cu at (96.3, 41.9)
- added R18: 10K, Resistor_SMD:R_0603_1608Metric, F.Cu at (96.3, 44.5)
- added R19: ?, Resistor_SMD:R_0603_1608Metric, F.Cu at (96.3, 47.0)
- added R2: 100K, Resistor_SMD:R_0603_1608Metric, F.Cu at (88.3, 49.5)
- added R20: ?, Resistor_SMD:R_0603_1608Metric, F.Cu at (96.3, 49.5)
- added R21: 10K, Resistor_SMD:R_0603_1608Metric, F.Cu at (96.3, 52.0)
- added R3: 10K, Resistor_SMD:R_0603_1608Metric, F.Cu at (88.3, 52.0)
- added R6: 220R, Resistor_SMD:R_0603_1608Metric, F.Cu at (88.3, 54.5)
- added R7: 220R, Resistor_SMD:R_0603_1608Metric, F.Cu at (92.3, 36.9)
- added R8: 220R, Resistor_SMD:R_0603_1608Metric, F.Cu at (92.3, 39.4)
- added R9: 10K, Resistor_SMD:R_0603_1608Metric, F.Cu at (92.3, 41.9)
Connections:
- Q6 pad 1: unconnected-(Q6-S-Pad1) -> LIPO-
- Q6 pad 2: unconnected-(Q6-S-Pad2) -> LIPO-
- Q6 pad 3: unconnected-(Q6-S-Pad3) -> LIPO-
- Q6 pad 4: unconnected-(Q6-G-Pad4) -> /Decharge
- Q6 pad 5: unconnected-(Q6-D-Pad5) -> /capa_out
- Q8 pad 1: /ST_ShortCUT -> Net-(Q8-G)
- Q9 pad 1: /ST_H30_LIPO -> Net-(Q9-G)

Commit message: Add files via upload
Parts:
- removed U3: STM32L476RCTx, Package_QFP:LQFP-64_10x10mm_P0.5mm
- added C10: 47nF, Capacitor_SMD:C_0603_1608Metric, F.Cu at (20.6, 52.3)
- added C13: 4.7uF, Capacitor_SMD:C_0603_1608Metric, F.Cu at (20.6, 54.8)
- added C14: 100nf, Capacitor_SMD:C_0603_1608Metric, F.Cu at (24.6, 29.7)
- added C15: 100nf, Capacitor_SMD:C_0603_1608Metric, F.Cu at (24.6, 32.2)
- added C16: 100nf, Capacitor_SMD:C_0603_1608Metric, F.Cu at (24.6, 34.7)
- added C17: 100nf, Capacitor_SMD:C_0603_1608Metric, F.Cu at (24.6, 37.2)
- added C18: 100nf, Capacitor_SMD:C_0603_1608Metric, F.Cu at (24.6, 39.8)
- added C19: 1uF, Capacitor_SMD:C_0603_1608Metric, F.Cu at (24.6, 42.3)
- added C20: 10nF, Capacitor_SMD:C_0603_1608Metric, F.Cu at (24.6, 44.8)
- added C21: 7.2pF, Capacitor_SMD:C_0603_1608Metric, F.Cu at (24.6, 47.3)
- added C212: 100n, Capacitor_SMD:C_0603_1608Metric, F.Cu at (28.6, 29.7)
- added C213: 100n, Capacitor_SMD:C_0603_1608Metric, F.Cu at (28.6, 32.2)
- added C22: 7.2pF, Capacitor_SMD:C_0603_1608Metric, F.Cu at (24.6, 49.8)
- added C23: 100nf, Capacitor_SMD:C_0603_1608Metric, F.Cu at (24.6, 52.3)
- added C65: 0.1uF, Capacitor_SMD:C_0603_1608Metric, F.Cu at (24.6, 54.8)
- added C7: 0.1uF, Capacitor_SMD:C_0603_1608Metric, F.Cu at (20.6, 44.8)
- added C8: 22uF, Capacitor_SMD:C_0603_1608Metric, F.Cu at (20.6, 47.3)
- added C9: 22uF, Capacitor_SMD:C_0603_1608Metric, F.Cu at (20.6, 49.8)
- added D10: RED, LED_SMD:LED_0603_1608Metric, F.Cu at (43.6, 68.9)
- added D11: STPS2L30A, STPS2L30A:DIOM5126X265N, F.Cu at (70.6, 48.5)
- added D201: 19-237/R6GHBHC-A01/2T, 19-237_R6GHBHC-A01_2T:19237R6GHBHCA012T, F.Cu at (79.1, 23.7)
- added D6: STPS2L30A, STPS2L30A:DIOM5126X265N, F.Cu at (70.6, 35.1)
- added D7: STPS2L30A, STPS2L30A:DIOM5126X265N, F.Cu at (70.6, 39.6)
- added D8: SS34, Diode_SMD:D_SMA, F.Cu at (71.3, 81.6)
- added D9: STPS2L30A, STPS2L30A:DIOM5126X265N, F.Cu at (70.6, 44.0)
- added F1: MF-MSMF200_12X-2, MF-MSMF200_12X-2:MFMSMF20012X2, F.Cu at (37.8, 59.2)
- added FB200: 600 @ 600 MHz, Inductor_SMD:L_0805_2012Metric, F.Cu at (31.1, 83.5)
- added H1: MountingHole_Pad, MountingHole:MountingHole_3.2mm_M3_Pad_Via, F.Cu at (62.7, 32.4)
- added H2: MountingHole_Pad, MountingHole:MountingHole_3.2mm_M3_Pad_Via, F.Cu at (62.7, 40.4)
- added H3: MountingHole_Pad, MountingHole:MountingHole_3.2mm_M3_Pad_Via, F.Cu at (62.7, 48.3)
- added H4: MountingHole_Pad, MountingHole:MountingHole_3.2mm_M3_Pad_Via, F.Cu at (62.7, 56.3)
- added IC3: W25N01GVZEIG, W25N01GVZEIG:SON127P800X600X80-9N-D, F.Cu at (23.7, 81.2)
- added J12: USB_C_Receptacle_USB2.0_14P, USBC:USBC, F.Cu at (40.5, 75.9)
- added J2: 62000211622, Connector_THT_Wurth:J_Wurth_WR-WTB_62000211622, F.Cu at (77.5, 31.4)
- added J3: 62000411622, Connector_THT_Wurth:J_Wurth_WR-WTB_62000411622, F.Cu at (49.7, 38.2)
- added J4: 62000411622, Connector_THT_Wurth:J_Wurth_WR-WTB_62000411622, F.Cu at (49.7, 45.1)
- added J401: SWD, Connector_PinHeader_1.27mm:PinHeader_2x05_P1.27mm_Vertical_SMD, F.Cu at (71.4, 54.9)
- added J5: 62000411622, Connector_THT_Wurth:J_Wurth_WR-WTB_62000411622, F.Cu at (49.7, 52.0)
- added J6: 62000411622, Connector_THT_Wurth:J_Wurth_WR-WTB_62000411622, F.Cu at (49.7, 58.8)
- added J7: 62000611622, Connector_THT_Wurth:J_Wurth_WR-WTB_62000611622, F.Cu at (21.6, 73.4)
- added J8: 62000411622, Connector_THT_Wurth:J_Wurth_WR-WTB_62000411622, F.Cu at (49.7, 65.7)
- added JP1: ~, jumper_footprints:Jumper_0603, F.Cu at (76.2, 49.6)
- added JP2: ~, jumper_footprints:Jumper_0603, F.Cu at (79.7, 49.6)
- added L1: 6.8uH, SRP5020CC-6R8M:INDPM5752X200N, F.Cu at (37.3, 65.9)
- added PS1: LD39050PU33R, LD39050PU33R:SON95P300X300X100-7N-D, F.Cu at (31.5, 79.8)
- added Q12: SI2301-TP, SI2301:SOT95P237X125-3N, F.Cu at (78.8, 76.3)
- added Q13: XT60_YELLOW, XT60:AMASS_XT60PB-F, F.Cu at (67.8, 74.6)
- added Q14: AO3401A, Package_TO_SOT_SMD:SOT-23, F.Cu at (78.7, 57.6)
- added R206: 1k, Resistor_SMD:R_0603_1608Metric, F.Cu at (44.6, 39.8)
- added R207: 1k, Resistor_SMD:R_0603_1608Metric, F.Cu at (44.6, 42.3)
- added R208: 1k, Resistor_SMD:R_0603_1608Metric, F.Cu at (44.6, 44.8)
- added R22: 220R, Resistor_SMD:R_0603_1608Metric, F.Cu at (36.6, 32.2)
- added R23: ?, Resistor_SMD:R_0603_1608Metric, F.Cu at (36.6, 34.7)
- added R24: ?, Resistor_SMD:R_0603_1608Metric, F.Cu at (36.6, 37.2)
- added R25: 10K, Resistor_SMD:R_0603_1608Metric, F.Cu at (36.6, 39.8)
- added R26: ?, Resistor_SMD:R_0603_1608Metric, F.Cu at (36.6, 42.3)
- added R27: 220R, Resistor_SMD:R_0603_1608Metric, F.Cu at (36.6, 44.8)
- added R28: 10K, Resistor_SMD:R_0603_1608Metric, F.Cu at (36.6, 47.3)
- added R29: 47R, Resistor_SMD:R_0603_1608Metric, F.Cu at (36.6, 49.8)
- added R30: 2K2, Resistor_SMD:R_0603_1608Metric, F.Cu at (36.6, 52.3)
- added R31: 2K2, Resistor_SMD:R_0603_1608Metric, F.Cu at (36.6, 54.8)
- added R32: 10K, Resistor_SMD:R_0603_1608Metric, F.Cu at (40.6, 29.7)
- added R33: 5K1, Resistor_SMD:R_0603_1608Metric, F.Cu at (40.6, 32.2)
- added R34: 22, Resistor_SMD:R_0603_1608Metric, F.Cu at (40.6, 34.7)
- added R35: 5K1, Resistor_SMD:R_0603_1608Metric, F.Cu at (40.6, 37.2)
- added R36: 22, Resistor_SMD:R_0603_1608Metric, F.Cu at (40.6, 39.8)
- added R37: 22, Resistor_SMD:R_0603_1608Metric, F.Cu at (40.6, 42.3)
- added R38: 22, Resistor_SMD:R_0603_1608Metric, F.Cu at (40.6, 44.8)
- added R39: 22, Resistor_SMD:R_0603_1608Metric, F.Cu at (40.6, 47.3)
- added R40: 22, Resistor_SMD:R_0603_1608Metric, F.Cu at (40.6, 49.8)
- added R400: 22, Resistor_SMD:R_0603_1608Metric, F.Cu at (44.6, 47.3)
- added R401: 22, Resistor_SMD:R_0603_1608Metric, F.Cu at (44.6, 49.8)
- added R402: 22, Resistor_SMD:R_0603_1608Metric, F.Cu at (44.6, 52.3)
- added R403: 22, Resistor_SMD:R_0603_1608Metric, F.Cu at (44.6, 54.8)
- added R41: 22, Resistor_SMD:R_0603_1608Metric, F.Cu at (40.6, 52.3)
- added R42: 22, Resistor_SMD:R_0603_1608Metric, F.Cu at (40.6, 54.8)
- added R43: 22, Resistor_SMD:R_0603_1608Metric, F.Cu at (44.6, 29.7)
- added R44: 22, Resistor_SMD:R_0603_1608Metric, F.Cu at (44.6, 32.2)
- added R45: 22, Resistor_SMD:R_0603_1608Metric, F.Cu at (44.6, 34.7)
- added R46: 22, Resistor_SMD:R_0603_1608Metric, F.Cu at (44.6, 37.2)
- added SW1: SW_Nidec_CAS-120A1, 450404015514:450404015514, F.Cu at (52.4, 72.8)
- added SW2: SW_Nidec_CAS-120A1, 450404015514:450404015514, F.Cu at (52.4, 80.5)
- added SW4: ~, SKSGPAE010:SKSG, F.Cu at (79.1, 80.6)
- added TP1: V_USB, TestPoint:TestPoint_Pad_D2.0mm, F.Cu at (44.6, 58.1)
- added U1: STM32L476RCTx, Package_QFP:LQFP-64_10x10mm_P0.5mm, F.Cu at (25.8, 63.3)
- added U9: USBLC6-2SC6, Package_TO_SOT_SMD:SOT-23-6, F.Cu at (78.8, 53.1)
- added Y1: 16MHz, NX3225SA-16.000000MHZ-B3:NX3225SA16000000MHZB3, F.Cu at (77.8, 38.3)
- C1: value 47nF -> 1uF
- C2, C4: value 22uF -> 100nF
- C3: value 22nF -> 1uF
- C6: value 0.1uF -> 22nF
- D1: value B240A-E3_5AT -> STPS2L30A; footprint B240A-E3_5AT:DIOM5127X229N -> STPS2L30A:DIOM5126X265N
- D2: value SS34 -> RED; footprint Diode_SMD:D_SMA -> LED_SMD:LED_0603_1608Metric
- D3: value LED -> SMAT70A-13-F; footprint LED_SMD:LED_0603_1608Metric -> SMAT70A-13-F:DIOM5226X230N
- D4: value SMAT70A-13-F -> SMAJ24A; footprint SMAT70A-13-F:DIOM5226X230N -> SMAJ24A:DIOM4325X250N
- D5: value SMAJ24A -> GREEN; footprint SMAJ24A:DIOM4325X250N -> LED_SMD:LED_0603_1608Metric
- IC1: value LTC4359IMS8#PBF -> MP2338GTL-P; footprint LTC4359IMS8#PBF:SOP65P490X110-8N -> MP2338GTL:SOTFL50P160X60-8N
- IC2: value MP2338GTL-P -> LTC4359IMS8#PBF; footprint MP2338GTL:SOTFL50P160X60-8N -> LTC4359IMS8#PBF:SOP65P490X110-8N
- J1: value Conn_01x02_Socket -> 62000411622; footprint Connector_PinSocket_2.54mm:PinSocket_1x02_P2.54mm_Vertical -> Connector_THT_Wurth:J_Wurth_WR-WTB_62000411622
- Q1: value PSMNR56-25YLEX -> XT60_YELLOW; footprint PSMNR56-25YLEX:PSMNR5830YLHX -> XT60:AMASS_XT60PB-M
- Q10: value XT60_YELLOW -> SI2301-TP; footprint XT60:AMASS_XT60PB-M -> SI2301:SOT95P237X125-3N
- Q11: value XT60_YELLOW -> PSMNR56-25YLEX; footprint XT60:AMASS_XT60PB-F -> PSMNR56-25YLEX:PSMNR5830YLHX
- Q2, Q6: value PSMNR56-25YLEX -> SI2301-TP; footprint PSMNR56-25YLEX:PSMNR5830YLHX -> SI2301:SOT95P237X125-3N
- Q7, Q8, Q9: value SI2301-TP -> PSMNR56-25YLEX; footprint SI2301:SOT95P237X125-3N -> PSMNR56-25YLEX:PSMNR5830YLHX
- R1: value 1K -> 100K
- R10: value 90.9K -> 2.2K
- R11, R3: value 10K -> 2.2K
- R12: value 10K -> 1K
- R13, R17: value 2.2K -> 10K
- R14, R5: value 10K -> 220R
- R15: value ? -> 10K
- R19: value ? -> 0.1R
- R2: value 100K -> 10K
- R20: value ? -> 100K
- R6, R7: value 220R -> 10K
- R8: value 220R -> 90.9K
- moved C2 67.9 mm to (20.6, 32.2)
- moved C3 67.9 mm to (20.6, 34.7)
- moved C4 67.9 mm to (20.6, 37.2)
- moved C5 67.9 mm to (20.6, 39.8)
- moved C6 67.9 mm to (20.6, 42.3)
- moved D2 67.7 mm to (43.6, 63.7)
- moved R7 65.0 mm to (28.6, 49.8)
- moved R8 65.0 mm to (28.6, 52.3)
- moved R9 65.0 mm to (28.6, 54.8)
- moved R15 63.9 mm to (32.6, 42.3)
- moved R16 63.9 mm to (32.6, 44.8)
- moved R17 63.9 mm to (32.6, 47.3)
- moved R18 63.9 mm to (32.6, 49.8)
- moved R19 63.9 mm to (32.6, 52.3)
- moved R20 63.9 mm to (32.6, 54.8)
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Connections:
- C1 pad 1: LIPO+ -> +5V
- C1 pad 2: Net-(IC1-VSS) -> -ST
- C2 pad 1: +12V -> +5V
- C2 pad 2: -H30 -> -ST
- C3 pad 1: Net-(IC2-SS) -> +3V3
- C3 pad 2: -H30 -> -ST
- C4 pad 1: +5V -> +3V3
- C4 pad 2: -H30 -> -ST
- C5 pad 1: +5V -> Net-(D9-K)
- C6 pad 1: Net-(IC2-BST) -> Net-(IC1-SS)
- C6 pad 2: /SW -> -H30
- D2 pad 1: Net-(D2-K) -> /PG
- D2 pad 2: -H30 -> Net-(D2-A)
- D4 pad A: Net-(D4-PadA) -> Net-(D3-PadA)
- D4 pad C: +H30 -> Net-(IC2-VSS)
- IC1 pad 1: /LTC gate -> /PG
- IC1 pad 2: +H30 -> Net-(D9-K)
- IC1 pad 3: unconnected-(IC1-NC_1-Pad3) -> /SW
- IC1 pad 4: +H30 -> -H30
- IC1 pad 5: unconnected-(IC1-~{SHDN}-Pad5) -> Net-(IC1-BST)
- IC1 pad 6: Net-(IC1-VSS) -> /EN
- IC1 pad 7: unconnected-(IC1-NC_2-Pad7) -> Net-(IC1-SS)
- IC1 pad 8: LIPO+ -> Net-(IC1-FB)
- IC2 pad 1: /PG -> /LTC gate
- IC2 pad 2: +12V -> +H30
- IC2 pad 3: /SW -> unconnected-(IC2-NC_1-Pad3)
- IC2 pad 4: -H30 -> +H30
- IC2 pad 5: Net-(IC2-BST) -> unconnected-(IC2-~{SHDN}-Pad5)
- IC2 pad 6: /EN -> Net-(IC2-VSS)
- IC2 pad 7: Net-(IC2-SS) -> unconnected-(IC2-NC_2-Pad7)
- IC2 pad 8: Net-(IC2-FB) -> OUT+
- J1 pad 1: Net-(D2-K) -> -ST
- J1 pad 2: -H30 -> Net-(J1-Pad2)
- Q1 pad 1: +H30 -> -H30
- Q10 pad 1: -H30 -> Net-(Q10-G)
- Q10 pad 2: +H30 -> Net-(D6-K)
- Q11 pad 1: LIPO- -> Net-(Q11-S-Pad1)
- Q11 pad 2: LIPO+ -> Net-(Q11-S-Pad1)
- Q2 pad 1: +H30 -> Net-(Q2-G)
- Q2 pad 2: +H30 -> Net-(Q2-S)
- Q2 pad 3: +H30 -> -H30
- Q3 pad 4: /Gate_Q3_Q4 -> Net-(Q2-S)
- Q3 pad 5: LIPO- -> +H30
- Q4 pad 1: -H30 -> +H30
- Q4 pad 2: -H30 -> +H30
- Q4 pad 3: -H30 -> +H30
- Q4 pad 4: /Gate_Q3_Q4 -> /LTC gate
- Q4 pad 5: LIPO- -> OUT+
- Q5 pad 1: -H30 -> +H30
- Q5 pad 2: -H30 -> +H30
- Q5 pad 3: -H30 -> +H30
- Q5 pad 4: Net-(Q5-G) -> /LTC gate
- Q5 pad 5: +H30 -> OUT+
- Q6 pad 1: LIPO- -> Net-(Q6-G)
- Q6 pad 2: LIPO- -> /Gate_H30-OUT-
- Q6 pad 3: LIPO- -> -H30
- Q7 pad 1: Net-(Q7-G) -> -H30
- Q7 pad 2: +5V -> -H30
- Q7 pad 3: Net-(D2-K) -> -H30
- Q8 pad 1: Net-(Q8-G) -> -H30
- Q8 pad 2: Net-(Q5-G) -> -H30
- Q9 pad 1: Net-(Q9-G) -> OUT-
- Q9 pad 2: /Gate_Q3_Q4 -> OUT-
- Q9 pad 3: -H30 -> OUT-
- R1 pad 1: Net-(IC1-VSS) -> /PG
- R1 pad 2: -H30 -> +5V
- R10 pad 1: Net-(R10-Pad1) -> Net-(D2-A)
- R11 pad 1: -H30 -> Net-(D5-A)
- R11 pad 2: Net-(R10-Pad1) -> +5V
- R12 pad 1: /PG -> Net-(IC2-VSS)
- R12 pad 2: +5V -> -H30
- R13 pad 1: Net-(D3-A) -> /TIM3_CH3
- R13 pad 2: +5V -> -H30
- R14 pad 1: /EN -> /TIM3_CH3
- R14 pad 2: +12V -> Net-(Q6-G)
- R15 pad 1: Net-(R15-Pad1) -> +3V3
- R15 pad 2: LIPO- -> /Gate_H30-OUT-
- R16 pad 1: /capa_out -> +H30
- R17 pad 1: -H30 -> Net-(SW1-A)
- R17 pad 2: /EN -> OUT-
- R18 pad 1: unconnected-(R18-Pad1) -> Net-(Q9-G)
- R19 pad 1: Net-(R15-Pad1) -> Net-(D7-A)
- R19 pad 2: LIPO- -> /capa_out
- R2 pad 1: /Gate_Q3_Q4 -> /EN
- R2 pad 2: -H30 -> Net-(D9-K)
- R20 pad 1: Net-(R15-Pad1) -> Net-(Q9-G)
- R20 pad 2: LIPO- -> OUT-
- R21 pad 1: Net-(SW1-A) -> OUT-
- R21 pad 2: LIPO- -> Net-(Q10-D)
- R3 pad 1: +5V -> -H30
- R3 pad 2: /ST_EV -> /EN
- R4 pad 1: +3V3 -> /TIM1_CH1
- R4 pad 2: Net-(Q5-G) -> -H30
- R5 pad 1: +3V3 -> /TIM1_CH1
- R5 pad 2: /Gate_Q3_Q4 -> Net-(Q2-G)
- R6 pad 1: /ST_EV -> +3V3
- R6 pad 2: Net-(Q7-G) -> Net-(Q2-S)
- R7 pad 1: /ST_ShortCUT -> Net-(IC1-FB)
- R7 pad 2: Net-(Q8-G) -> Net-(R7-Pad2)
- R8 pad 1: /ST_H30_LIPO -> Net-(R7-Pad2)
- R8 pad 2: Net-(Q9-G) -> +5V
- R9 pad 1: Net-(IC2-FB) -> -H30
- R9 pad 2: Net-(R10-Pad1) -> Net-(R7-Pad2)

Commit message: Add files via upload
Parts:
- removed C212, C213: 100n, Capacitor_SMD:C_0603_1608Metric
- removed C65: 0.1uF, Capacitor_SMD:C_0603_1608Metric
- removed D201: 19-237/R6GHBHC-A01/2T, 19-237_R6GHBHC-A01_2T:19237R6GHBHCA012T
- removed FB200: 600 @ 600 MHz, Inductor_SMD:L_0805_2012Metric
- removed J401: SWD, Connector_PinHeader_1.27mm:PinHeader_2x05_P1.27mm_Vertical_SMD
- removed Q13: XT60_YELLOW, XT60:AMASS_XT60PB-F
- removed Q14: AO3401A, Package_TO_SOT_SMD:SOT-23
- removed R206, R207, R208: 1k, Resistor_SMD:R_0603_1608Metric
- removed R400, R401, R402, R403: 22, Resistor_SMD:R_0603_1608Metric
- removed SW4: ~, SKSGPAE010:SKSG
- removed U9: USBLC6-2SC6, Package_TO_SOT_SMD:SOT-23-6
- added C11: 100nf, Capacitor_SMD:C_0603_1608Metric, F.Cu at (73.7, 80.7)
- added C12: 100nf, Capacitor_SMD:C_0603_1608Metric, F.Cu at (73.7, 83.2)
- added C24: 470 uF, Capacitor_THT_Wurth_PT:CP_Wurth_WCAP-PTHT-P5D10L12.5, F.Cu at (95.3, 105.4)
- added C25: 1uF, Capacitor_SMD:C_0603_1608Metric, F.Cu at (77.7, 80.7)
- added C26: 470 uF, Capacitor_THT_Wurth_PT:CP_Wurth_WCAP-PTHT-P5D10L12.5, F.Cu at (95.3, 117.5)
- added C27: 100nF, Capacitor_SMD:C_0603_1608Metric, F.Cu at (77.7, 83.2)
- added C28: 470 uF, Capacitor_THT_Wurth_PT:CP_Wurth_WCAP-PTHT-P5D10L12.5, F.Cu at (95.3, 129.5)
- added C29: 10 uF, Capacitor_SMD_Wurth:CP_Wurth_WCAP-ASLI-D4L5.5, F.Cu at (135.3, 121.7)
- added C30: 10 uF, Capacitor_SMD_Wurth:CP_Wurth_WCAP-ASLI-D4L5.5, F.Cu at (135.3, 128.0)
- added C31: 10 uF, Capacitor_SMD_Wurth:CP_Wurth_WCAP-ASLI-D4L5.5, F.Cu at (135.3, 134.3)
- added C32: 2.2uF, Capacitor_SMD:C_0603_1608Metric, F.Cu at (77.7, 85.7)
- added C33: 100nF, Capacitor_SMD:C_0603_1608Metric, F.Cu at (77.7, 88.2)
- added C34: 100nF, Capacitor_SMD:C_0603_1608Metric, F.Cu at (81.8, 58.1)
- added C35: C, Capacitor_SMD:C_0603_1608Metric, F.Cu at (81.8, 60.6)
- added D12: BLUE, LED_SMD:LED_0603_1608Metric, F.Cu at (63.7, 127.8)
- added D13: BAT54S-HF, BAT54S-HF:SOT95P240X115-3N, F.Cu at (114.2, 120.8)
- added D14: BAT54S-HF, BAT54S-HF:SOT95P240X115-3N, F.Cu at (114.2, 125.3)
- added D15: BAT54S-HF, BAT54S-HF:SOT95P240X115-3N, F.Cu at (114.2, 129.8)
- added D16: SS34, Diode_SMD:D_SMA, F.Cu at (138.4, 114.8)
- added D17: BAT54S-HF, BAT54S-HF:SOT95P240X115-3N, F.Cu at (119.1, 120.8)
- added D18: BAT54S-HF, BAT54S-HF:SOT95P240X115-3N, F.Cu at (119.1, 125.3)
- added D19: BAT54S-HF, BAT54S-HF:SOT95P240X115-3N, F.Cu at (119.1, 129.8)
- added D20: BAT54S-HF, BAT54S-HF:SOT95P240X115-3N, F.Cu at (124.0, 120.8)
- added D21: BAT54S-HF, BAT54S-HF:SOT95P240X115-3N, F.Cu at (124.0, 125.3)
- added D22: BAT54S-HF, BAT54S-HF:SOT95P240X115-3N, F.Cu at (124.0, 129.8)
- added D23: BAT54S-HF, BAT54S-HF:SOT95P240X115-3N, F.Cu at (128.8, 120.8)
- added D24: BAT54S-HF, BAT54S-HF:SOT95P240X115-3N, F.Cu at (128.8, 125.3)
- added D25: BAT54S-HF, BAT54S-HF:SOT95P240X115-3N, F.Cu at (128.8, 129.8)
- added FB1: 600 @ 600 MHz, Inductor_SMD:L_0805_2012Metric, F.Cu at (138.9, 81.0)
- added IC4: ADS1115IDGSR, ADS1115IDGSR:SOP50P490X110-10N, F.Cu at (107.5, 81.4)
- added IC5: ADS1115IDGSR, ADS1115IDGSR:SOP50P490X110-10N, F.Cu at (107.5, 86.1)
- added IC6: DRV8833CPWPR, DRV8833CPWPR:SOP65P640X120-17N, F.Cu at (125.8, 135.6)
- added IC7: LM358DR, LM358DR:SOIC127P600X175-8N, F.Cu at (138.6, 102.7)
- added J10: 62000211622, Connector_THT_Wurth:J_Wurth_WR-WTB_62000211622, F.Cu at (86.8, 109.1)
- added J11: 62000611622, Connector_THT_Wurth:J_Wurth_WR-WTB_62000611622, F.Cu at (127.9, 85.5)
- added J13: 62000211622, Connector_THT_Wurth:J_Wurth_WR-WTB_62000211622, F.Cu at (86.8, 116.0)
- added J14: 62000211622, Connector_THT_Wurth:J_Wurth_WR-WTB_62000211622, F.Cu at (86.8, 122.9)
- added J15: 62000211622, Connector_THT_Wurth:J_Wurth_WR-WTB_62000211622, F.Cu at (86.8, 129.8)
- added J16: 62000211622, Connector_THT_Wurth:J_Wurth_WR-WTB_62000211622, F.Cu at (86.8, 136.6)
- added J17: 62000311622, Connector_THT_Wurth:J_Wurth_WR-WTB_62000311622, F.Cu at (64.7, 59.7)
- added J18: 62000311622, Connector_THT_Wurth:J_Wurth_WR-WTB_62000311622, F.Cu at (64.7, 66.6)
- added J19: 62000311622, Connector_THT_Wurth:J_Wurth_WR-WTB_62000311622, F.Cu at (64.7, 73.5)
- added J20: 62000311622, Connector_THT_Wurth:J_Wurth_WR-WTB_62000311622, F.Cu at (64.7, 80.3)
- added J21: 62000311622, Connector_THT_Wurth:J_Wurth_WR-WTB_62000311622, F.Cu at (64.7, 87.2)
- added J22: 62000311622, Connector_THT_Wurth:J_Wurth_WR-WTB_62000311622, F.Cu at (64.7, 94.1)
- added J23: 62000311622, Connector_THT_Wurth:J_Wurth_WR-WTB_62000311622, F.Cu at (64.7, 101.0)
- added J24: 62000311622, Connector_THT_Wurth:J_Wurth_WR-WTB_62000311622, F.Cu at (64.7, 107.8)
- added J9: 62000411622, Connector_THT_Wurth:J_Wurth_WR-WTB_62000411622, F.Cu at (74.8, 126.7)
- added JP3: ~, jumper_footprints:Jumper_3points_0402, F.Cu at (138.4, 92.4)
- added JP4: ~, jumper_footprints:Jumper_3points_0402, F.Cu at (138.4, 96.2)
- added NT1: NetTie_2, NetTie:NetTie-2_SMD_Pad2.0mm, F.Cu at (139.2, 63.1)
- added R47: 220R, Resistor_SMD:R_0603_1608Metric, F.Cu at (93.8, 80.7)
- added R48: 22, Resistor_SMD:R_0603_1608Metric, F.Cu at (93.8, 83.2)
- added R49: 22, Resistor_SMD:R_0603_1608Metric, F.Cu at (93.8, 85.7)
- added R50: 22, Resistor_SMD:R_0603_1608Metric, F.Cu at (93.8, 88.2)
- added R51: 22, Resistor_SMD:R_0603_1608Metric, F.Cu at (97.8, 58.1)
- added R52: 22, Resistor_SMD:R_0603_1608Metric, F.Cu at (97.8, 60.6)
- added R53: 22, Resistor_SMD:R_0603_1608Metric, F.Cu at (97.8, 63.1)
- added R54: 2k2, Resistor_SMD:R_0603_1608Metric, F.Cu at (97.8, 65.6)
- added R55: 10K, Resistor_SMD:R_0603_1608Metric, F.Cu at (97.8, 68.1)
- added R56: 10K, Resistor_SMD:R_0603_1608Metric, F.Cu at (97.8, 70.7)
- added R57: 10K, Resistor_SMD:R_0603_1608Metric, F.Cu at (97.8, 73.2)
- added R58: 220R, Resistor_SMD:R_0603_1608Metric, F.Cu at (97.8, 75.7)
- added R59: 15K, Resistor_SMD:R_0603_1608Metric, F.Cu at (97.8, 78.2)
- added R60: 220R, Resistor_SMD:R_0603_1608Metric, F.Cu at (97.8, 80.7)
- added R61: 2k2, Resistor_SMD:R_0603_1608Metric, F.Cu at (97.8, 83.2)
- added R62: 10K, Resistor_SMD:R_0603_1608Metric, F.Cu at (97.8, 85.7)
- added R63: 12K, Resistor_SMD:R_0603_1608Metric, F.Cu at (97.8, 88.2)
- added R64: ?, Resistor_SMD:R_0603_1608Metric, F.Cu at (101.8, 58.1)
- added R65: ?, Resistor_SMD:R_0603_1608Metric, F.Cu at (101.8, 60.6)
- added R66: 22, Resistor_SMD:R_0603_1608Metric, F.Cu at (101.8, 63.1)
- added R67: 22, Resistor_SMD:R_0603_1608Metric, F.Cu at (101.8, 65.6)
- added R68: 22, Resistor_SMD:R_0603_1608Metric, F.Cu at (101.8, 68.1)
- added R69: 22, Resistor_SMD:R_0603_1608Metric, F.Cu at (101.8, 70.7)
- added R70: 22, Resistor_SMD:R_0603_1608Metric, F.Cu at (101.8, 73.2)
- added R71: 22, Resistor_SMD:R_0603_1608Metric, F.Cu at (101.8, 75.7)
- added R72: 22, Resistor_SMD:R_0603_1608Metric, F.Cu at (101.8, 78.2)
- added R73: 22, Resistor_SMD:R_0603_1608Metric, F.Cu at (101.8, 80.7)
- added SW3: SW_Nidec_CAS-120A1, Button_Switch_SMD:Nidec_Copal_CAS-120A, F.Cu at (133.8, 93.0)
- added TP2: NFAULT, TestPoint:TestPoint_Pad_D2.0mm, F.Cu at (67.8, 124.8)
- added U2: USBLC6-2SC6, Package_TO_SOT_SMD:SOT-23-6, F.Cu at (138.3, 67.0)
- added U3: LTC1044, LTC1044:SOIC127P600X175-8N, F.Cu at (138.6, 109.2)
- C1, C3: value 1uF -> 7.2pF
- C10: value 47nF -> 22nF
- C13: value 4.7uF -> 0.1uF
- C14: value 100nf -> 1uF
- C15, C17: value 100nf -> 22uF
- C16: value 100nf -> 10nF
- C18: value 100nf -> 47nF
- C19: value 1uF -> 0.1uF
- C2: value 100nF -> 100nf
- C20: value 10nF -> 1uF
- C21: value 7.2pF -> 100nF
- C22: value 7.2pF -> 100n
- C23: value 100nf -> 100n
- C4: value 100nF -> 220 uF; footprint Capacitor_SMD:C_0603_1608Metric -> Capacitor_SMD_Wurth:CP_Wurth_WCAP-ASLI-D8L10.5
- C5: value 22uF -> 4.7uF
- C6: value 22nF -> 22uF
- C7: value 0.1uF -> 100nf
- C8, C9: value 22uF -> 100nf
- D1, D6: value STPS2L30A -> RED; footprint STPS2L30A:DIOM5126X265N -> LED_SMD:LED_0603_1608Metric
- D10, D2: value RED -> STPS2L30A; footprint LED_SMD:LED_0603_1608Metric -> STPS2L30A:DIOM5126X265N
- D3: value SMAT70A-13-F -> STPS2L30A; footprint SMAT70A-13-F:DIOM5226X230N -> STPS2L30A:DIOM5126X265N
- D4: value SMAJ24A -> SMAT70A-13-F; footprint SMAJ24A:DIOM4325X250N -> SMAT70A-13-F:DIOM5226X230N
- D5: value GREEN -> SMAJ24A; footprint LED_SMD:LED_0603_1608Metric -> SMAJ24A:DIOM4325X250N
- D7: value STPS2L30A -> GREEN; footprint STPS2L30A:DIOM5126X265N -> LED_SMD:LED_0603_1608Metric
- D8: value SS34 -> 19-237/R6GHBHC-A01/2T; footprint Diode_SMD:D_SMA -> 19-237_R6GHBHC-A01_2T:19237R6GHBHCA012T
- J1: value 62000411622 -> USB_C_Receptacle_USB2.0_14P; footprint Connector_THT_Wurth:J_Wurth_WR-WTB_62000411622 -> USBC:USBC
- J12: value USB_C_Receptacle_USB2.0_14P -> 62000411622; footprint USBC:USBC -> Connector_THT_Wurth:J_Wurth_WR-WTB_62000411622
- J2: value 62000211622 -> SWD; footprint Connector_THT_Wurth:J_Wurth_WR-WTB_62000211622 -> Connector_PinHeader_1.27mm:PinHeader_2x07_P1.27mm_Vertical_SMD
- J6: value 62000411622 -> 62000211622; footprint Connector_THT_Wurth:J_Wurth_WR-WTB_62000411622 -> Connector_THT_Wurth:J_Wurth_WR-WTB_62000211622
- J7: value 62000611622 -> 62000411622; footprint Connector_THT_Wurth:J_Wurth_WR-WTB_62000611622 -> Connector_THT_Wurth:J_Wurth_WR-WTB_62000411622
- Q10: value SI2301-TP -> PSMNR56-25YLEX; footprint SI2301:SOT95P237X125-3N -> PSMNR56-25YLEX:PSMNR5830YLHX
- Q11: value PSMNR56-25YLEX -> XT60_YELLOW; footprint PSMNR56-25YLEX:PSMNR5830YLHX -> XT60:AMASS_XT60PB-F
- Q2: value SI2301-TP -> AO3401A; footprint SI2301:SOT95P237X125-3N -> Package_TO_SOT_SMD:SOT-23
- Q3, Q8: value PSMNR56-25YLEX -> SI2301-TP; footprint PSMNR56-25YLEX:PSMNR5830YLHX -> SI2301:SOT95P237X125-3N
- R1: value 100K -> 10K
- R11: value 2.2K -> 10K
- R12: value 1K -> 90.9K
- R14: value 220R -> 2K2
- R15: value 10K -> 2K2
- R16, R17: value 10K -> 2.2K
- R18: value 10K -> 1K
- R19: value 0.1R -> 1k
- R20: value 100K -> 1k
- R21: value 10K -> 1k
- R22, R27, R5: value 220R -> 10K
- R23, R24: value ? -> 5K1
- R25, R6: value 10K -> 220R
- R26: value ? -> 10K
- R29: value 47R -> 10K
- R3: value 2.2K -> 47R
- R30: value 2K2 -> 10K
- R31: value 2K2 -> 22
- R32: value 10K -> 22
- R33: value 5K1 -> 100K
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Connections:
- C1 pad 1: +5V -> /HSE_IN
- C10 pad 1: OUT+ -> Net-(IC1-SS)
- C10 pad 2: Net-(IC2-VSS) -> -H30
- C13 pad 1: +3V3 -> Net-(IC1-BST)
- C13 pad 2: -ST -> /SW
- C14 pad 1: +3V3 -> +3V3A
- C15 pad 1: +3V3 -> +5V
- C15 pad 2: -ST -> -H30
- C16 pad 1: +3V3 -> +3V3A
- C17 pad 1: +3V3 -> +5V
- C17 pad 2: -ST -> -H30
- C18 pad 1: +3V3 -> OUT+
- C18 pad 2: -ST -> Net-(IC2-VSS)
- C19 pad 1: +3V3A -> +VBUS
- C2 pad 1: +5V -> /NRST
- C20 pad 1: +3V3A -> +5V
- C21 pad 1: /HSE_IN -> +5V
- C22 pad 1: Net-(C22-Pad1) -> +3V3
- C23 pad 1: /NRST -> +3V3
- C3 pad 1: +3V3 -> Net-(C3-Pad1)
- C4 pad 1: +3V3 -> Net-(D2-K)
- C4 pad 2: -ST -> -H30
- C5 pad 1: Net-(D9-K) -> +3V3
- C5 pad 2: -H30 -> -ST
- C6 pad 1: Net-(IC1-SS) -> Net-(D2-K)
- C7 pad 1: Net-(IC1-BST) -> +3V3
- C7 pad 2: /SW -> -ST
- C8 pad 1: +5V -> +3V3
- C8 pad 2: -H30 -> -ST
- C9 pad 1: +5V -> +3V3
- C9 pad 2: -H30 -> -ST
- D1 pad 1: +12V -> -ST
- D1 pad 2: +H30 -> Net-(D1-A)
- D10 pad 1: -ST -> Net-(D10-K)
- D11 pad 1: +5V -> Net-(D10-K)
- D11 pad 2: +VBUS -> Net-(D11-A)
- D2 pad 1: /PG -> Net-(D2-K)
- D2 pad 2: Net-(D2-A) -> +VBUS
- D4 pad A: Net-(D3-PadA) -> Net-(D4-PadA)
- D4 pad C: Net-(IC2-VSS) -> +H30
- D6 pad 1: Net-(D6-K) -> /PG
- D7 pad 1: Net-(D6-K) -> -H30
- D8 pad 1: Net-(D8-K) -> Net-(D8-RK)
- D8 pad 2: -H30 -> Net-(D8-GK)
- D9 pad 1: Net-(D9-K) -> +5V
- F1 pad 2: Net-(Q14-D) -> Net-(Q2-D)
- IC1 pad 2: Net-(D9-K) -> Net-(D2-K)
- J2 pad 1: -H30 -> unconnected-(J2-Pin_1-Pad1)
- J2 pad 2: Net-(D8-K) -> unconnected-(J2-Pin_2-Pad2)
- J7 pad 2: /SPI1_SCK -> Net-(J7-Pad2)
- J7 pad 3: /SPI1_MISO -> Net-(J7-Pad3)
- J7 pad 4: /SPI1_MOSI -> +3V3
- Q10 pad 1: Net-(Q10-G) -> OUT-
- Q10 pad 2: Net-(D6-K) -> OUT-
- Q10 pad 3: Net-(Q10-D) -> OUT-
- Q11 pad 1: Net-(Q11-S-Pad1) -> OUT-
- Q11 pad 2: Net-(Q11-S-Pad1) -> OUT+
- Q12 pad 3: Net-(D8-K) -> Net-(D16-K)
- Q2 pad 1: Net-(Q2-G) -> -H30
- Q2 pad 2: Net-(Q2-S) -> Net-(D2-K)
- Q2 pad 3: -H30 -> Net-(Q2-D)
- Q3 pad 1: -H30 -> Net-(Q3-G)
- Q3 pad 2: -H30 -> Net-(Q3-S)
- Q4 pad 1: +H30 -> -H30
- Q4 pad 2: +H30 -> -H30
- Q4 pad 3: +H30 -> -H30
- Q4 pad 4: /LTC gate -> Net-(Q3-S)
- Q4 pad 5: OUT+ -> +H30
- Q8 pad 1: -H30 -> Net-(Q8-G)
- Q8 pad 2: -H30 -> Net-(D10-K)
- Q8 pad 3: -H30 -> Net-(Q8-D)
- R1 pad 1: /PG -> /NRST
- R1 pad 2: +5V -> +3V3
- R10 pad 1: Net-(D2-A) -> -H30
- R10 pad 2: +5V -> /EN
- R11 pad 1: Net-(D5-A) -> Net-(IC1-FB)
- R11 pad 2: +5V -> Net-(R11-Pad2)
- R12 pad 1: Net-(IC2-VSS) -> Net-(R11-Pad2)
- R12 pad 2: -H30 -> +5V
- R13 pad 1: /TIM3_CH3 -> -H30
- R13 pad 2: -H30 -> Net-(R11-Pad2)
- R14 pad 1: /TIM3_CH3 -> /I2C1_SCL
- R14 pad 2: Net-(Q6-G) -> +3V3
- R15 pad 1: +3V3 -> /I2C1_SCA
- R15 pad 2: /Gate_H30-OUT- -> +3V3
- R16 pad 1: +H30 -> Net-(D6-A)
- R16 pad 2: Net-(D6-A) -> +5V
- R17 pad 1: Net-(SW1-A) -> Net-(D7-A)
- R17 pad 2: OUT- -> +5V
- R18 pad 1: Net-(Q9-G) -> Net-(IC2-VSS)
- R18 pad 2: +H30 -> -H30
- R19 pad 1: Net-(D7-A) -> Net-(D8-RK)
- R19 pad 2: /capa_out -> /TIM2_CH1
- R2 pad 1: /EN -> Net-(D1-A)
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Other:
- board outline added: 81.2 x 116.5 mm

Commit message: upload V1
Parts:
- added C36: 2.2uF, Capacitor_SMD:C_0603_1608Metric, F.Cu at (92.9, 90.5)
- added C37: 100nF, Capacitor_SMD:C_0603_1608Metric, F.Cu at (92.9, 93.0)
- added C38: 100nF, Capacitor_SMD:C_0603_1608Metric, F.Cu at (92.9, 95.6)
- added C39: C, Capacitor_SMD:C_0603_1608Metric, F.Cu at (92.9, 98.1)
- added D26: BAT54S-HF, BAT54S-HF:SOT95P240X115-3N, F.Cu at (99.9, 123.7)
- added D27: BAT54S-HF, BAT54S-HF:SOT95P240X115-3N, F.Cu at (99.9, 128.3)
- added Q13: XT60_YELLOW, XT60:AMASS_XT60PB-F, F.Cu at (111.5, 131.2)
- added Q14: SI2301-TP, SI2301:SOT95P237X125-3N, F.Cu at (130.6, 133.0)
- added R74: 22, Resistor_SMD:R_0603_1608Metric, F.Cu at (117.0, 103.1)
- added R75: 22, Resistor_SMD:R_0603_1608Metric, F.Cu at (117.0, 105.6)
- added R76: 22, Resistor_SMD:R_0603_1608Metric, F.Cu at (117.0, 108.1)
- added R77: 22, Resistor_SMD:R_0603_1608Metric, F.Cu at (117.0, 110.6)
- added R78: 22, Resistor_SMD:R_0603_1608Metric, F.Cu at (117.0, 113.1)
- added TP3: NFAULT, TestPoint:TestPoint_Pad_D2.0mm, F.Cu at (129.5, 111.3)
- C25: value 1uF -> 100nF
- C26: value 470 uF -> 1uF; footprint Capacitor_THT_Wurth_PT:CP_Wurth_WCAP-PTHT-P5D10L12.5 -> Capacitor_SMD:C_0603_1608Metric
- C27: value 100nF -> 470 uF; footprint Capacitor_SMD:C_0603_1608Metric -> Capacitor_THT_Wurth_PT:CP_Wurth_WCAP-PTHT-P5D10L12.5
- C28: value 470 uF -> 100nF; footprint Capacitor_THT_Wurth_PT:CP_Wurth_WCAP-PTHT-P5D10L12.5 -> Capacitor_SMD:C_0603_1608Metric
- C29, C30, C31: value 10 uF -> 470 uF; footprint Capacitor_SMD_Wurth:CP_Wurth_WCAP-ASLI-D4L5.5 -> Capacitor_THT_Wurth_PT:CP_Wurth_WCAP-PTHT-P5D10L12.5
- C32: value 2.2uF -> 470 uF; footprint Capacitor_SMD:C_0603_1608Metric -> Capacitor_THT_Wurth_PT:CP_Wurth_WCAP-PTHT-P5D10L12.5
- C33, C34: value 100nF -> 10 uF; footprint Capacitor_SMD:C_0603_1608Metric -> Capacitor_SMD_Wurth:CP_Wurth_WCAP-ASLI-D4L5.5
- C35: value C -> 10 uF; footprint Capacitor_SMD:C_0603_1608Metric -> Capacitor_SMD_Wurth:CP_Wurth_WCAP-ASLI-D4L5.5
- C4: value 220 uF -> 47 uF; footprint Capacitor_SMD_Wurth:CP_Wurth_WCAP-ASLI-D8L10.5 -> Capacitor_SMD_Wurth:CP_Wurth_WCAP-ASLI-D6.3L5.5
- D12: value BLUE -> STPS2L30A; footprint LED_SMD:LED_0603_1608Metric -> STPS2L30A:DIOM5126X265N
- D13: value BAT54S-HF -> RED; footprint BAT54S-HF:SOT95P240X115-3N -> LED_SMD:LED_0603_1608Metric
- D14: value BAT54S-HF -> BLUE; footprint BAT54S-HF:SOT95P240X115-3N -> LED_SMD:LED_0603_1608Metric
- D16: value SS34 -> BAT54S-HF; footprint Diode_SMD:D_SMA -> BAT54S-HF:SOT95P240X115-3N
- D18: value BAT54S-HF -> SS34; footprint BAT54S-HF:SOT95P240X115-3N -> Diode_SMD:D_SMA
- D3: value STPS2L30A -> RED; footprint STPS2L30A:DIOM5126X265N -> LED_SMD:LED_0603_1608Metric
- D4: value SMAT70A-13-F -> STPS2L30A; footprint SMAT70A-13-F:DIOM5226X230N -> STPS2L30A:DIOM5126X265N
- D5: value SMAJ24A -> SMAT70A-13-F; footprint SMAJ24A:DIOM4325X250N -> SMAT70A-13-F:DIOM5226X230N
- D6: value RED -> SMAJ24A; footprint LED_SMD:LED_0603_1608Metric -> SMAJ24A:DIOM4325X250N
- D7: value GREEN -> RED
- D8: value 19-237/R6GHBHC-A01/2T -> GREEN; footprint 19-237_R6GHBHC-A01_2T:19237R6GHBHCA012T -> LED_SMD:LED_0603_1608Metric
- D9: value STPS2L30A -> 19-237/R6GHBHC-A01/2T; footprint STPS2L30A:DIOM5126X265N -> 19-237_R6GHBHC-A01_2T:19237R6GHBHCA012T
- Q11: value XT60_YELLOW -> 2N7002; footprint XT60:AMASS_XT60PB-F -> Package_TO_SOT_SMD:SOT-23
- Q12, Q6, Q8: value SI2301-TP -> PSMNR56-25YLEX; footprint SI2301:SOT95P237X125-3N -> PSMNR56-25YLEX:PSMNR5830YLHX
- Q4: value PSMNR56-25YLEX -> 2N7002; footprint PSMNR56-25YLEX:PSMNR5830YLHX -> Package_TO_SOT_SMD:SOT-23
- Q7, Q9: value PSMNR56-25YLEX -> SI2301-TP; footprint PSMNR56-25YLEX:PSMNR5830YLHX -> SI2301:SOT95P237X125-3N
- R11: value 10K -> 100K
- R12: value 90.9K -> 10K
- R13: value 10K -> 2.2K
- R14: value 2K2 -> 10K
- R15: value 2K2 -> 90.9K
- R16: value 2.2K -> 10K
- R17: value 2.2K -> 2K2
- R18: value 1K -> 2K2
- R19, R20: value 1k -> 2.2K
- R21: value 1k -> 1K
- R22: value 10K -> 1k
- R23, R24: value 5K1 -> 1k
- R25, R60: value 220R -> 10K
- R26, R27: value 10K -> 5K1
- R28: value 10K -> 220R
- R31, R32, R41, R67: value 22 -> 10K
- R33: value 100K -> 10K
- R34: value 22 -> 100K
- R38, R55, R56, R57: value 10K -> 22
- R42, R43, R47, R58: value 220R -> 22
- R45, R49, R52: value 22 -> 220R
- R50: value 22 -> 220
- R51: value 22 -> 2.2K
- R54: value 2k2 -> 22
- R59: value 15K -> 2k2
- R61: value 2k2 -> 10K
- R63: value 12K -> 220R
- R64: value ? -> 15K
- R65: value ? -> 220R
- R66: value 22 -> 2k2
- R68: value 22 -> 12K
- R69, R70: value 22 -> ?
- R8: value 100K -> 220R
- R9: value 10K -> 220
- TP2: value NFAULT -> Gate_H30->OUT
- moved U2 98.5 mm to (59.3, 125.7)
- moved JP3 90.3 mm to (54.7, 126.3)
- moved JP4 90.3 mm to (54.7, 130.0)
- moved J2 90.0 mm to (67.6, 126.3)
- moved D4 88.9 mm to (123.0, 69.3)
- moved C35 83.7 mm to (124.1, 132.8)
- moved C34 80.4 mm to (124.1, 126.4)
- moved IC6 79.4 mm to (128.5, 56.2)
- moved D12 74.5 mm to (123.0, 82.7)
- moved Y1 73.9 mm to (134.9, 108.0)
- moved D1 71.4 mm to (135.1, 118.2)
- moved D7 71.4 mm to (135.1, 123.4)
- moved C31 70.2 mm to (110.5, 68.7)
- moved J1 68.8 mm to (68.5, 101.6)
- moved Q6 65.7 mm to (87.5, 57.8)
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Connections:
- C24 pad 2: /capa_out -> Net-(Q10-D)
- C25 pad 1: +3V3 -> Net-(Q10-G)
- C25 pad 2: -ST -> OUT-
- C26 pad 1: OUT+ -> +3V3
- C26 pad 2: /capa_out -> -ST
- C27 pad 1: +3V3 -> OUT+
- C27 pad 2: -ST -> Net-(Q10-D)
- C28 pad 1: OUT+ -> +3V3
- C28 pad 2: /capa_out -> -ST
- C29 pad 1: Net-(U3-CAP+) -> OUT+
- C29 pad 2: Net-(U3-CAP-) -> Net-(Q10-D)
- C30 pad 1: -ST -> OUT+
- C30 pad 2: -12V -> Net-(Q10-D)
- C31 pad 1: +12V -> OUT+
- C31 pad 2: -H30 -> Net-(Q10-D)
- C32 pad 1: /VINT -> OUT+
- C32 pad 2: -H30 -> Net-(Q10-D)
- C33 pad 1: +5V -> Net-(U3-CAP+)
- C33 pad 2: -ST -> Net-(U3-CAP-)
- C34 pad 1: +5V -> -ST
- C34 pad 2: -ST -> -12V
- C35 pad 1: Net-(IC7-IN1-) -> +12V
- C35 pad 2: Net-(IC7-OUT1) -> -H30
- D10 pad 1: Net-(D10-K) -> +5V
- D10 pad 2: Net-(D10-A) -> +VBUS
- D11 pad 1: Net-(D10-K) -> Net-(D11-K)
- D12 pad 1: Net-(D12-K) -> Net-(D11-K)
- D12 pad 2: +5V -> Net-(D12-A)
- D13 pad 1: -ST -> Net-(D13-K)
- D13 pad 2: +3V3 -> Net-(D13-A)
- D14 pad 1: -ST -> Net-(D14-K)
- D14 pad 2: +3V3 -> +5V
- D15 pad 3: /ADC2_EX0 -> /ADC1_IN1+
- D16 pad 1: Net-(D16-K) -> -ST
- D16 pad 2: -H30 -> +3V3
- D17 pad 3: /ADC3_IN3+ -> /ADC2_EX0
- D18 pad 1: -ST -> Net-(D18-K)
- D18 pad 2: +3V3 -> -H30
- D19 pad 3: /ADC2_EX1 -> /ADC3_IN3+
- D20 pad 3: /ADC1_IN2- -> /ADC1_EX1
- D21 pad 3: /ADC1_EX2 -> /ADC2_EX1
- D22 pad 3: /ADC2_EX2 -> /ADC1_IN2-
- D23 pad 3: /ADC2_IN4 -> /ADC1_EX2
- D24 pad 3: /ADC1_EX3 -> /ADC2_EX2
- D25 pad 3: /ADC2_EX3 -> /ADC2_IN4
- D3 pad 1: +12V -> Net-(D3-K)
- D3 pad 2: +H30 -> Net-(D3-A)
- D5 pad A: Net-(D4-PadA) -> Net-(D5-PadA)
- D5 pad C: Net-(IC2-VSS) -> +H30
- D7 pad 1: -H30 -> /PG
- D8 pad 1: Net-(D8-RK) -> -H30
- D8 pad 2: Net-(D8-GK) -> Net-(D8-A)
- D9 pad 1: +5V -> Net-(D9-RK)
- D9 pad 2: +VBUS -> Net-(D9-GK)
- J13 pad 2: Net-(D16-K) -> Net-(D18-K)
- Q11 pad 1: OUT- -> Net-(Q11-G)
- Q11 pad 2: OUT+ -> -H30
- Q12 pad 1: Net-(Q12-G) -> OUT-
- Q12 pad 2: +5V -> OUT-
- Q12 pad 3: Net-(D16-K) -> OUT-
- Q3 pad 2: Net-(Q3-S) -> /LED_Short
- Q4 pad 1: -H30 -> Net-(Q4-G)
- Q4 pad 3: -H30 -> Net-(D3-K)
- Q5 pad 1: +H30 -> -H30
- Q5 pad 2: +H30 -> -H30
- Q5 pad 3: +H30 -> -H30
- Q5 pad 4: /LTC gate -> Net-(Q5-G)
- Q5 pad 5: OUT+ -> +H30
- Q6 pad 1: Net-(Q6-G) -> +H30
- Q6 pad 2: /Gate_H30-OUT- -> +H30
- Q6 pad 3: -H30 -> +H30
- Q7 pad 1: -H30 -> Net-(Q7-G)
- Q7 pad 2: -H30 -> /Gate_H30-OUT-
- Q8 pad 1: Net-(Q8-G) -> -H30
- Q8 pad 2: Net-(D10-K) -> -H30
- Q8 pad 3: Net-(Q8-D) -> -H30
- Q9 pad 1: OUT- -> Net-(Q9-G)
- Q9 pad 2: OUT- -> Net-(D11-K)
- Q9 pad 3: OUT- -> /LED_Capa
- R10 pad 1: -H30 -> +3V3
- R10 pad 2: /EN -> Net-(D3-A)
- R11 pad 1: Net-(IC1-FB) -> /PG
- R11 pad 2: Net-(R11-Pad2) -> +5V
- R12 pad 1: Net-(R11-Pad2) -> /EN
- R12 pad 2: +5V -> Net-(D2-K)
- R13 pad 2: Net-(R11-Pad2) -> /EN
- R14 pad 1: /I2C1_SCL -> Net-(IC1-FB)
- R14 pad 2: +3V3 -> Net-(R14-Pad2)
- R15 pad 1: /I2C1_SCA -> Net-(R14-Pad2)
- R15 pad 2: +3V3 -> +5V
- R16 pad 1: Net-(D6-A) -> -H30
- R16 pad 2: +5V -> Net-(R14-Pad2)
- R17 pad 1: Net-(D7-A) -> /I2C1_SCL
- R17 pad 2: +5V -> +3V3
- R18 pad 1: Net-(IC2-VSS) -> /I2C1_SCA
- R18 pad 2: -H30 -> +3V3
- R19 pad 1: Net-(D8-RK) -> Net-(D7-A)
- R19 pad 2: /TIM2_CH1 -> +5V
- R20 pad 1: /TIM2_CH3 -> Net-(D8-A)
- R20 pad 2: Net-(D8-GK) -> +5V
- R21 pad 1: Net-(D8-BK) -> Net-(IC2-VSS)
- R21 pad 2: /TIM2_CH4 -> -H30
- R22 pad 1: /TIM3_CH3 -> Net-(D9-RK)
- R22 pad 2: -H30 -> /TIM2_CH1
- R23 pad 1: GND -> /TIM2_CH3
- R23 pad 2: Net-(J1-CC1) -> Net-(D9-GK)
- R24 pad 1: GND -> Net-(D9-BK)
- R24 pad 2: Net-(J1-CC2) -> /TIM2_CH4
- R25 pad 2: Net-(Q6-G) -> -H30
- R26 pad 1: +3V3 -> GND
- R26 pad 2: /Gate_H30-OUT- -> Net-(J1-CC1)
- R27 pad 1: +H30 -> GND
- R27 pad 2: Net-(D10-A) -> Net-(J1-CC2)
- R28 pad 1: Net-(SW3-A) -> /TIM3_CH3
- R28 pad 2: OUT- -> Net-(Q7-G)
- R29 pad 1: /capa_out -> +3V3
- R29 pad 2: Net-(D11-A) -> /Gate_H30-OUT-
- R30 pad 1: Net-(Q9-G) -> +H30
- R30 pad 2: +H30 -> Net-(D11-A)
- R31 pad 1: Net-(J3-Pad3) -> Net-(SW3-A)
- R31 pad 2: /USART3_RX -> OUT-
- R32 pad 1: Net-(J3-Pad2) -> Net-(Q10-G)
- R32 pad 2: /USART3_TX -> +H30
- R33 pad 1: Net-(Q9-G) -> /capa_out
- R33 pad 2: OUT- -> Net-(D12-A)
- R34 pad 1: Net-(J4-Pad3) -> Net-(Q10-G)
- R34 pad 2: /ADC1_IN1+ -> OUT-
- R35 pad 1: Net-(J4-Pad2) -> Net-(J3-Pad3)
- R35 pad 2: /ADC1_IN2- -> /USART3_RX
- R36 pad 1: Net-(J5-Pad3) -> Net-(J3-Pad2)
- R36 pad 2: /I2C1_SCA -> /USART3_TX
- R37 pad 1: Net-(J5-Pad2) -> Net-(J4-Pad3)
- R37 pad 2: /I2C1_SCL -> /ADC1_IN1+
- R38 pad 1: OUT- -> Net-(J4-Pad2)
- R38 pad 2: Net-(Q8-D) -> /ADC1_IN2-
- R39 pad 1: /SWDIO -> Net-(J5-Pad3)
- R39 pad 2: Net-(J2-Pin_4) -> /I2C1_SCA
- R40 pad 1: /NRST -> Net-(J5-Pad2)
- R40 pad 2: Net-(J2-Pin_12) -> /I2C1_SCL
- R41 pad 1: /SWCLK -> OUT-
- R41 pad 2: Net-(J2-Pin_6) -> /LED_Capa
- R42 pad 1: Net-(Q8-D) -> /SWDIO
- R42 pad 2: Net-(Q10-G) -> Net-(J2-Pin_4)
- R43 pad 1: /capa_out -> /NRST
- R43 pad 2: Net-(Q10-D) -> Net-(J2-Pin_12)
- R44 pad 1: /SWO -> /SWCLK
- R44 pad 2: Net-(J2-Pin_8) -> Net-(J2-Pin_6)
- R45 pad 1: Net-(J7-Pad3) -> /LED_Capa
- R45 pad 2: /UART4_RX -> Net-(Q12-G)
- R46 pad 1: Net-(J7-Pad2) -> /SWO
- R46 pad 2: /UART4_TX -> Net-(J2-Pin_8)
- R47 pad 1: /capa_out -> Net-(J7-Pad3)
- R47 pad 2: Net-(Q10-D) -> /UART4_RX
- R48 pad 1: Net-(J8-Pad3) -> Net-(J7-Pad2)
- R48 pad 2: /ADC3_IN3+ -> /UART4_TX
- R49 pad 1: Net-(J8-Pad2) -> Net-(Q10-D)
- R49 pad 2: /ADC2_IN4 -> /capa_out
- R50 pad 1: Net-(J9-Pad3) -> /LED_Capa
- R50 pad 2: /I2C1_SCA -> Net-(Q11-G)
- R51 pad 1: Net-(J9-Pad2) -> +3V3
- R51 pad 2: /I2C1_SCL -> Net-(D13-A)
- R52 pad 1: Net-(J12-Pad3) -> Net-(Q10-D)
- R52 pad 2: /UART5_RX -> /capa_out
- R53 pad 1: Net-(J12-Pad2) -> Net-(J8-Pad3)
- R53 pad 2: /UART5_TX -> /ADC3_IN3+
- R54 pad 1: Net-(D12-K) -> Net-(J8-Pad2)
- R54 pad 2: /TIM3_CH1 -> /ADC2_IN4
- R55 pad 1: +3V3 -> Net-(J9-Pad3)
- R55 pad 2: /ALERT1 -> /I2C1_SCA
- R56 pad 1: +3V3 -> Net-(J9-Pad2)
- R56 pad 2: /ALERT2 -> /I2C1_SCL
- R57 pad 1: +5V -> Net-(J12-Pad3)
- R57 pad 2: /TIM3_CH1 -> /UART5_RX
- R58 pad 1: /TIM3_CH1 -> Net-(J12-Pad2)
- R58 pad 2: Net-(Q12-G) -> /UART5_TX
- R59 pad 1: -12V -> Net-(D14-K)
- R59 pad 2: Net-(IC7-IN2-) -> /TIM3_CH1
- R60 pad 1: Net-(IC7-IN1-) -> +3V3
- R60 pad 2: Net-(IC7-OUT1) -> /ALERT1
- R61 pad 1: Net-(IC7-IN2-) -> +3V3
- R61 pad 2: /ADC2_IN4 -> /ALERT2
- R62 pad 1: +3V3 -> +5V
- R62 pad 2: /NFAULT -> /TIM3_CH1
- R63 pad 1: Net-(IC7-IN2-) -> /TIM3_CH1
- R63 pad 2: Net-(IC7-OUT1) -> Net-(Q14-G)
- R64 pad 1: /AISEN -> -12V
- R64 pad 2: -H30 -> Net-(IC7-IN2-)
- R65 pad 1: /BISEN -> Net-(IC7-IN1-)
- R65 pad 2: -H30 -> Net-(IC7-OUT1)
- R66 pad 1: Net-(J17-Pad2) -> Net-(IC7-IN2-)
- R66 pad 2: /ADC1_EX0 -> /ADC2_IN4
- R67 pad 1: Net-(J18-Pad2) -> +3V3
- R67 pad 2: /ADC1_EX1 -> /NFAULT
- R68 pad 1: Net-(J19-Pad2) -> Net-(IC7-IN2-)
- R68 pad 2: /ADC1_EX2 -> Net-(IC7-OUT1)
- R69 pad 1: Net-(J20-Pad2) -> /AISEN
- R69 pad 2: /ADC1_EX3 -> -H30
- R7 pad 2: Net-(Q3-S) -> /LED_Short
- R70 pad 1: Net-(J21-Pad2) -> /BISEN
- R70 pad 2: /ADC2_EX0 -> -H30
- R71 pad 1: Net-(J22-Pad2) -> Net-(J17-Pad2)
- R71 pad 2: /ADC2_EX1 -> /ADC1_EX0
- R72 pad 1: Net-(J23-Pad2) -> Net-(J18-Pad2)
- R72 pad 2: /ADC2_EX2 -> /ADC1_EX1
- R73 pad 1: Net-(J24-Pad2) -> Net-(J19-Pad2)
- R73 pad 2: /ADC2_EX3 -> /ADC1_EX2
- R8 pad 1: /PG -> /LED_Short
- R8 pad 2: +5V -> Net-(Q5-G)
- R9 pad 1: /EN -> /LED_Short
- R9 pad 2: Net-(D2-K) -> Net-(Q4-G)
- SW3 pad 1: Net-(D10-K) -> Net-(D11-K)
- SW3 pad 2: Net-(Q8-G) -> Net-(Q9-G)
- TP2 pad 1: /NFAULT -> /Gate_H30-OUT-
