File: PCB/H30_controler_board.kicad_pcb (KiCad board)
At the start: 2 copper layers, 81.2 x 116.5 mm, 212 parts, among them IC1 MP2338GTL-P, IC2 LTC4359IMS8#PBF, IC3 W25N01GVZEIG, IC4 ADS1115IDGSR, IC5 ADS1115IDGSR, IC6 DRV8833CPWPR, IC7 LM358DR, J1 USB_C_Receptacle_USB2.0_14P, J10 62000211622, J11 62000611622, J12 62000411622, J13 62000211622, J14 62000211622, J15 62000211622, J16 62000211622, J17 62000311622, J18 62000311622, J19 62000311622, J2 SWD, J20 62000311622, J21 62000311622, J22 62000311622, J23 62000311622, J24 62000311622, J3 62000411622, J4 62000411622, J5 62000411622, J6 62000211622, J7 62000411622, J8 62000411622, J9 62000411622, Q1 XT60_YELLOW, Q10 PSMNR56-25YLEX, Q11 2N7002, Q12 PSMNR56-25YLEX, Q13 XT60_YELLOW, Q14 SI2301-TP, Q2 AO3401A, Q3 SI2301-TP, Q4 2N7002, Q5 PSMNR56-25YLEX, Q6 PSMNR56-25YLEX, Q7 SI2301-TP, Q8 PSMNR56-25YLEX, Q9 SI2301-TP, SW1 SW_Nidec_CAS-120A1, SW3 SW_Nidec_CAS-120A1, U1 STM32L476RCTx, U2 USBLC6-2SC6, U3 LTC1044, Y1 16MHz

Commit message: Add files via upload
Parts:
- removed Q14: SI2301-TP, SI2301:SOT95P237X125-3N
- added D28: BAT54S-HF, BAT54S-HF:SOT95P240X115-3N, F.Cu at (64.1, 92.1)
- added J25: 653003114822, Connector_THT_Wurth:J_Wurth_WR-WTB_653003114822, F.Cu at (108.2, 109.4)
- added J26: 653003114822, Connector_THT_Wurth:J_Wurth_WR-WTB_653003114822, F.Cu at (108.2, 114.8)
- added J27: 653003114822, Connector_THT_Wurth:J_Wurth_WR-WTB_653003114822, F.Cu at (108.2, 120.2)
- added LS1: CMT-8530S-SMT-TR, CMT-8530S-SMT-TR:CMT8530SSMTTR, F.Cu at (109.8, 38.6)
- added R79: 22, Resistor_SMD:R_0603_1608Metric, F.Cu at (77.2, 69.4)
- added R80: 22, Resistor_SMD:R_0603_1608Metric, F.Cu at (77.2, 71.9)
- added R81: 0R, Resistor_SMD:R_0603_1608Metric, F.Cu at (77.2, 74.4)
- added TP4: V_USB, TestPoint:TestPoint_Pad_D1.5mm, F.Cu at (66.9, 99.7)
- added TP5: Gate_H30->OUT, TestPoint:TestPoint_Pad_D1.5mm, F.Cu at (70.5, 96.1)
- added TP6: V_Reverse, TestPoint:TestPoint_Pad_D1.5mm, F.Cu at (70.5, 99.7)
- added TP7: V_Reverse, TestPoint:TestPoint_Pad_D1.5mm, F.Cu at (74.0, 96.1)
- added TP8: NFAULT, TestPoint:TestPoint_Pad_D1.5mm, F.Cu at (74.0, 99.7)
- D10: value STPS2L30A -> 19-237/R6GHBHC-A01/2T; footprint STPS2L30A:DIOM5126X265N -> 19-237_R6GHBHC-A01_2T:19237R6GHBHCA012T
- D13, D3: value RED -> STPS2L30A; footprint LED_SMD:LED_0603_1608Metric -> STPS2L30A:DIOM5126X265N
- D14: value BLUE -> RED
- D15: value BAT54S-HF -> BLUE; footprint BAT54S-HF:SOT95P240X115-3N -> LED_SMD:LED_0603_1608Metric
- D18: value SS34 -> BAT54S-HF; footprint Diode_SMD:D_SMA -> BAT54S-HF:SOT95P240X115-3N
- D19: value BAT54S-HF -> SS34; footprint BAT54S-HF:SOT95P240X115-3N -> Diode_SMD:D_SMA
- D2, D4: value STPS2L30A -> RED; footprint STPS2L30A:DIOM5126X265N -> LED_SMD:LED_0603_1608Metric
- D5: value SMAT70A-13-F -> STPS2L30A; footprint SMAT70A-13-F:DIOM5226X230N -> STPS2L30A:DIOM5126X265N
- D6: value SMAJ24A -> SMAT70A-13-F; footprint SMAJ24A:DIOM4325X250N -> SMAT70A-13-F:DIOM5226X230N
- D7: value RED -> SMAJ24A; footprint LED_SMD:LED_0603_1608Metric -> SMAJ24A:DIOM4325X250N
- D8: value GREEN -> RED
- D9: value 19-237/R6GHBHC-A01/2T -> GREEN; footprint 19-237_R6GHBHC-A01_2T:19237R6GHBHCA012T -> LED_SMD:LED_0603_1608Metric
- H3: value MountingHole_Pad -> Pad 3.2 mm M3
- J1: value USB_C_Receptacle_USB2.0_14P -> XT60_YELLOW; footprint USBC:USBC -> XT60:AMASS_XT60PB-M
- J10, J13, J6: value 62000211622 -> 653004114822; footprint Connector_THT_Wurth:J_Wurth_WR-WTB_62000211622 -> Connector_THT_Wurth:J_Wurth_WR-WTB_653004114822
- J11: value 62000611622 -> 653004114822; footprint Connector_THT_Wurth:J_Wurth_WR-WTB_62000611622 -> Connector_THT_Wurth:J_Wurth_WR-WTB_653004114822
- J12, J7: value 62000411622 -> 653002114822; footprint Connector_THT_Wurth:J_Wurth_WR-WTB_62000411622 -> Connector_THT_Wurth:J_Wurth_WR-WTB_653002114822
- J14: value 62000211622 -> 653006114822; footprint Connector_THT_Wurth:J_Wurth_WR-WTB_62000211622 -> Connector_THT_Wurth:J_Wurth_WR-WTB_653006114822
- J15: value 62000211622 -> XT60_YELLOW; footprint Connector_THT_Wurth:J_Wurth_WR-WTB_62000211622 -> XT60:AMASS_XT60PB-F
- J16: value 62000211622 -> 653002114822; footprint Connector_THT_Wurth:J_Wurth_WR-WTB_62000211622 -> Connector_THT_Wurth:J_Wurth_WR-WTB_653002114822
- J17, J18, J19: value 62000311622 -> 653002114822; footprint Connector_THT_Wurth:J_Wurth_WR-WTB_62000311622 -> Connector_THT_Wurth:J_Wurth_WR-WTB_653002114822
- J2: value SWD -> USB_C_Receptacle_USB2.0_14P; footprint Connector_PinHeader_1.27mm:PinHeader_2x07_P1.27mm_Vertical_SMD -> USBC:USBC
- J20, J21, J22, J23, J24: value 62000311622 -> 653003114822; footprint Connector_THT_Wurth:J_Wurth_WR-WTB_62000311622 -> Connector_THT_Wurth:J_Wurth_WR-WTB_653003114822
- J3: value 62000411622 -> SWD; footprint Connector_THT_Wurth:J_Wurth_WR-WTB_62000411622 -> Connector_PinHeader_1.27mm:PinHeader_2x07_P1.27mm_Vertical_SMD
- J4, J5, J9: value 62000411622 -> 653004114822; footprint Connector_THT_Wurth:J_Wurth_WR-WTB_62000411622 -> Connector_THT_Wurth:J_Wurth_WR-WTB_653004114822
- J8: value 62000411622 -> TC2030; footprint Connector_THT_Wurth:J_Wurth_WR-WTB_62000411622 -> Connector:Tag-Connect_TC2030-IDC-NL_2x03_P1.27mm_Vertical
- Q1: value XT60_YELLOW -> AO3401A; footprint XT60:AMASS_XT60PB-M -> Package_TO_SOT_SMD:SOT-23
- Q13: value XT60_YELLOW -> SI2301-TP; footprint XT60:AMASS_XT60PB-F -> SI2301:SOT95P237X125-3N
- Q2: value AO3401A -> SI2301-TP; footprint Package_TO_SOT_SMD:SOT-23 -> SI2301:SOT95P237X125-3N
- Q3: value SI2301-TP -> 2N7002; footprint SI2301:SOT95P237X125-3N -> Package_TO_SOT_SMD:SOT-23
- Q4: value 2N7002 -> PSMNR56-25YLEX; footprint Package_TO_SOT_SMD:SOT-23 -> PSMNR56-25YLEX:PSMNR5830YLHX
- Q6: value PSMNR56-25YLEX -> SI2301-TP; footprint PSMNR56-25YLEX:PSMNR5830YLHX -> SI2301:SOT95P237X125-3N
- Q7: value SI2301-TP -> PSMNR56-25YLEX; footprint SI2301:SOT95P237X125-3N -> PSMNR56-25YLEX:PSMNR5830YLHX
- Q8: value PSMNR56-25YLEX -> 2N7002; footprint PSMNR56-25YLEX:PSMNR5830YLHX -> Package_TO_SOT_SMD:SOT-23
- R10: value 2.2K -> 220
- R11: value 100K -> 2.2K
- R12: value 10K -> 100K
- R13: value 2.2K -> 10K
- R14: value 10K -> 2.2K
- R15: value 90.9K -> 10K
- R16: value 10K -> 90.9K
- R17: value 2K2 -> 10K
- R19: value 2.2K -> 2K2
- R2: value 10K -> 5K1
- R21: value 1K -> 2.2K
- R22: value 1k -> 1K
- R25: value 10K -> 1k
- R26: value 5K1 -> 10K
- R28: value 220R -> 5K1
- R29, R7: value 10K -> 220R
- R3: value 47R -> 10K
- R31: value 10K -> 0
- R32: value 10K -> 220
- R34: value 100K -> 10K
- R35, R36, R48: value 22 -> 10K
- R37: value 22 -> 100K
- R4: value 10K -> 47R
- R41, R60, R61: value 10K -> 22
- R45: value 220R -> 22
- R50: value 220 -> 22
- R51: value 2.2K -> 22
- R53: value 22 -> 220
- R54: value 22 -> 2.2K
- R55: value 22 -> 220R
- R59: value 2k2 -> 22
- R6, R63, R65, R8: value 220R -> 10K
- R62: value 10K -> 2k2
- R64: value 15K -> 10K
- R66: value 2k2 -> 220R
- R67: value 10K -> 15K
- R68: value 12K -> 220R
- R69: value ? -> 2k2
- R70: value ? -> 10K
- R71: value 22 -> 12K
- R72: value 22 -> 0R
- R9: value 220 -> 220R
- TP1: value V_USB -> SDA; footprint TestPoint:TestPoint_Pad_D2.0mm -> TestPoint:TestPoint_Pad_D1.5mm
- TP2: value Gate_H30->OUT -> SCL; footprint TestPoint:TestPoint_Pad_D2.0mm -> TestPoint:TestPoint_Pad_D1.5mm
- TP3: value NFAULT -> LTC gate; footprint TestPoint:TestPoint_Pad_D2.0mm -> TestPoint:TestPoint_Pad_D1.5mm
- moved H2 170.8 mm to (232.7, 41.6)
- moved H3 164.8 mm to (232.7, 64.6)
- moved H4 105.1 mm to (159.7, 64.6)
- moved H1 104.5 mm to (159.7, 41.6)
- moved JP3 96.1 mm to (125.8, 61.6)
- moved JP4 96.1 mm to (125.8, 65.3)
- moved IC3 87.5 mm to (60.6, 123.9)
- moved L1 82.1 mm to (119.6, 62.1)
- moved D6 78.1 mm to (125.5, 71.7)
- moved SW3 76.0 mm to (69.8, 104.9)
- moved SW1 76.0 mm to (64.3, 104.9)
- moved R42 75.3 mm to (69.2, 46.8)
- moved R43 75.3 mm to (69.2, 49.3)
- moved J17 73.8 mm to (115.7, 98.7)
- moved D5 73.6 mm to (123.4, 86.2)
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Connections:
- C4 pad 1: Net-(D2-K) -> Net-(D3-K)
- C6 pad 1: Net-(D2-K) -> Net-(D3-K)
- D1 pad 1: -ST -> Net-(D1-K)
- D10 pad 1: +5V -> Net-(D10-RK)
- D10 pad 2: +VBUS -> Net-(D10-GK)
- D11 pad 1: Net-(D11-K) -> +5V
- D11 pad 2: Net-(D11-A) -> +VBUS
- D12 pad 1: Net-(D11-K) -> Net-(D12-K)
- D13 pad 1: Net-(D13-K) -> Net-(D12-K)
- D14 pad 2: +5V -> Net-(D14-A)
- D15 pad 1: -ST -> Net-(D15-K)
- D15 pad 2: +3V3 -> +5V
- D16 pad 3: /ADC1_EX0 -> /ADC1_IN1+
- D17 pad 3: /ADC2_EX0 -> /ADC1_EX0
- D18 pad 1: Net-(D18-K) -> -ST
- D18 pad 2: -H30 -> +3V3
- D19 pad 1: -ST -> Net-(D19-K)
- D19 pad 2: +3V3 -> -H30
- D2 pad 1: Net-(D2-K) -> -ST
- D2 pad 2: +VBUS -> Net-(D2-A)
- D20 pad 3: /ADC1_EX1 -> /ADC3_IN3+
- D21 pad 3: /ADC2_EX1 -> /ADC1_EX1
- D22 pad 3: /ADC1_IN2- -> /ADC2_EX1
- D23 pad 3: /ADC1_EX2 -> /ADC1_IN2-
- D24 pad 3: /ADC2_EX2 -> /ADC1_EX2
- D25 pad 3: /ADC2_IN4 -> /ADC2_EX2
- D26 pad 3: /ADC1_EX3 -> /ADC2_IN4
- D27 pad 3: /ADC2_EX3 -> /ADC1_EX3
- D3 pad 2: Net-(D3-A) -> +VBUS
- D4 pad 1: +12V -> Net-(D4-K)
- D4 pad 2: +H30 -> Net-(D4-A)
- D6 pad A: Net-(D5-PadA) -> Net-(D6-PadA)
- D6 pad C: Net-(IC2-VSS) -> +H30
- D8 pad 1: -H30 -> /PG
- D9 pad 1: Net-(D9-RK) -> -H30
- D9 pad 2: Net-(D9-GK) -> Net-(D9-A)
- F1 pad 2: Net-(Q2-D) -> Net-(D1-K)
- IC1 pad 2: Net-(D2-K) -> Net-(D3-K)
- IC4 pad 9: /I2C1_SCA -> /I2C1_SDA
- IC5 pad 9: /I2C1_SCA -> /I2C1_SDA
- IC6 pad 14: unconnected-(IC6-VINT-Pad14) -> /VINT
- J11 pad 2: /SPI1_SCK -> Net-(J11-Pad2)
- J11 pad 3: /SPI1_MISO -> Net-(J11-Pad3)
- J11 pad 4: /SPI1_MOSI -> +3V3
- J13 pad 1: -H30 -> -ST
- J13 pad 2: Net-(D18-K) -> Net-(J13-Pad2)
- J14 pad 2: Net-(IC7-IN1-) -> /SPI1_SCK
- J15 pad 1: Net-(IC6-AOUT2) -> OUT-
- J15 pad 2: Net-(IC6-AOUT1) -> OUT+
- J16 pad 1: Net-(IC6-BOUT2) -> -H30
- J16 pad 2: Net-(IC6-BOUT1) -> Net-(D19-K)
- J17 pad 2: Net-(J17-Pad2) -> Net-(IC7-IN1-)
- J18 pad 1: -ST -> Net-(IC6-AOUT2)
- J18 pad 2: Net-(J18-Pad2) -> Net-(IC6-AOUT1)
- J19 pad 1: -ST -> Net-(IC6-BOUT1)
- J19 pad 2: Net-(J19-Pad2) -> Net-(IC6-BOUT2)
- J22 pad 1: unconnected-(J22-Pad1) -> -ST
- J3 pad 1: -ST -> unconnected-(J3-Pin_1-Pad1)
- J3 pad 2: Net-(J3-Pad2) -> unconnected-(J3-Pin_2-Pad2)
- J3 pad 3: Net-(J3-Pad3) -> +3V3
- J3 pad 4: +3V3 -> Net-(J3-Pin_4)
- J8 pad 1: -ST -> +3V3
- J8 pad 2: Net-(J8-Pad2) -> /SWDIO
- J8 pad 3: Net-(J8-Pad3) -> /NRST
- J8 pad 4: +3V3 -> /SWCLK
- JP3 pad 3: Net-(J6-Pad2) -> Net-(J7-Pad2)
- JP4 pad 3: Net-(J10-Pad2) -> Net-(J12-Pad2)
- Q1 pad 2: +H30 -> Net-(D3-K)
- Q11 pad 3: Net-(D13-K) -> Net-(D14-K)
- Q13 pad 1: OUT- -> Net-(Q13-G)
- Q13 pad 2: OUT+ -> +5V
- Q2 pad 1: -H30 -> Net-(Q2-G)
- Q2 pad 2: Net-(D2-K) -> /LED_Short
- Q2 pad 3: Net-(Q2-D) -> -H30
- Q3 pad 2: /LED_Short -> -H30
- Q3 pad 3: -H30 -> Net-(D4-K)
- Q4 pad 1: Net-(Q4-G) -> -H30
- Q4 pad 3: Net-(D3-K) -> -H30
- Q5 pad 1: -H30 -> +H30
- Q5 pad 2: -H30 -> +H30
- Q5 pad 3: -H30 -> +H30
- Q5 pad 4: Net-(Q5-G) -> /LTC gate
- Q5 pad 5: +H30 -> OUT+
- Q6 pad 1: +H30 -> Net-(Q6-G)
- Q6 pad 2: +H30 -> /Gate_H30-OUT-
- Q6 pad 3: +H30 -> -H30
- Q7 pad 1: Net-(Q7-G) -> -H30
- Q7 pad 2: /Gate_H30-OUT- -> -H30
- Q8 pad 1: -H30 -> Net-(Q8-G)
- Q8 pad 2: -H30 -> -ST
- Q8 pad 3: -H30 -> Net-(Q8-D)
- Q9 pad 2: Net-(D11-K) -> Net-(D12-K)
- R10 pad 1: +3V3 -> /LED_Short
- R10 pad 2: Net-(D3-A) -> Net-(Q3-G)
- R11 pad 1: /PG -> +3V3
- R11 pad 2: +5V -> Net-(D4-A)
- R12 pad 1: /EN -> /PG
- R12 pad 2: Net-(D2-K) -> +5V
- R13 pad 1: -H30 -> /EN
- R13 pad 2: /EN -> Net-(D3-K)
- R14 pad 1: Net-(IC1-FB) -> -H30
- R14 pad 2: Net-(R14-Pad2) -> /EN
- R15 pad 1: Net-(R14-Pad2) -> Net-(IC1-FB)
- R15 pad 2: +5V -> Net-(R15-Pad2)
- R16 pad 1: -H30 -> Net-(R15-Pad2)
- R16 pad 2: Net-(R14-Pad2) -> +5V
- R17 pad 1: /I2C1_SCL -> -H30
- R17 pad 2: +3V3 -> Net-(R15-Pad2)
- R18 pad 1: /I2C1_SCA -> /I2C1_SCL
- R19 pad 1: Net-(D7-A) -> /I2C1_SDA
- R19 pad 2: +5V -> +3V3
- R2 pad 1: Net-(D1-A) -> +12V
- R2 pad 2: Net-(SW1-B) -> Net-(D1-A)
- R21 pad 1: Net-(IC2-VSS) -> Net-(D9-A)
- R21 pad 2: -H30 -> +5V
- R22 pad 1: Net-(D9-RK) -> Net-(IC2-VSS)
- R22 pad 2: /TIM2_CH1 -> -H30
- R23 pad 1: /TIM2_CH3 -> Net-(D10-RK)
- R23 pad 2: Net-(D9-GK) -> /TIM2_CH1
- R24 pad 1: Net-(D9-BK) -> /TIM2_CH3
- R24 pad 2: /TIM2_CH4 -> Net-(D10-GK)
- R25 pad 1: /TIM3_CH3 -> Net-(D10-BK)
- R25 pad 2: -H30 -> /TIM2_CH4
- R26 pad 1: GND -> /TIM3_CH3
- R26 pad 2: Net-(J1-CC1) -> -H30
- R27 pad 1: GND -> -ST
- R27 pad 2: Net-(J1-CC2) -> Net-(J2-CC1)
- R28 pad 1: /TIM3_CH3 -> -ST
- R28 pad 2: Net-(Q7-G) -> Net-(J2-CC2)
- R29 pad 1: +3V3 -> /TIM3_CH3
- R29 pad 2: /Gate_H30-OUT- -> Net-(Q6-G)
- R3 pad 1: Net-(C3-Pad1) -> Net-(D2-A)
- R3 pad 2: /HSE_OUT -> Net-(SW1-B)
- R30 pad 1: +H30 -> +3V3
- R30 pad 2: Net-(D11-A) -> /Gate_H30-OUT-
- R31 pad 1: Net-(SW3-A) -> Net-(Q8-D)
- R31 pad 2: OUT- -> Net-(LS1--)
- R32 pad 1: Net-(Q10-G) -> /TIM1_CH3
- R32 pad 2: +H30 -> Net-(Q8-G)
- R33 pad 1: /capa_out -> +H30
- R34 pad 1: Net-(Q10-G) -> Net-(SW3-A)
- R35 pad 1: Net-(J3-Pad3) -> Net-(Q10-G)
- R35 pad 2: /USART3_RX -> +H30
- R36 pad 1: Net-(J3-Pad2) -> /capa_out
- R36 pad 2: /USART3_TX -> Net-(D13-A)
- R37 pad 1: Net-(J4-Pad3) -> Net-(Q10-G)
- R37 pad 2: /ADC1_IN1+ -> OUT-
- R38 pad 1: Net-(J4-Pad2) -> Net-(J4-Pad3)
- R38 pad 2: /ADC1_IN2- -> /USART3_RX
- R39 pad 1: Net-(J5-Pad3) -> Net-(J4-Pad2)
- R39 pad 2: /I2C1_SCA -> /USART3_TX
- R4 pad 1: Net-(SW1-B) -> Net-(C3-Pad1)
- R4 pad 2: /BOOT0 -> /HSE_OUT
- R40 pad 1: Net-(J5-Pad2) -> /SWDIO
- R40 pad 2: /I2C1_SCL -> Net-(J3-Pin_4)
- R41 pad 1: OUT- -> /SWCLK
- R41 pad 2: /LED_Capa -> Net-(J3-Pin_6)
- R42 pad 1: /SWDIO -> /SWO
- R42 pad 2: Net-(J2-Pin_4) -> Net-(J3-Pin_8)
- R43 pad 2: Net-(J2-Pin_12) -> Net-(J3-Pin_12)
- R44 pad 1: /SWCLK -> Net-(J5-Pad3)
- R44 pad 2: Net-(J2-Pin_6) -> /ADC1_IN1+
- R45 pad 1: /LED_Capa -> Net-(J5-Pad2)
- R45 pad 2: Net-(Q12-G) -> /ADC1_IN2-
- R46 pad 1: /SWO -> Net-(J6-Pad3)
- R46 pad 2: Net-(J2-Pin_8) -> /I2C1_SDA
- R47 pad 1: Net-(J7-Pad3) -> Net-(J6-Pad2)
- R47 pad 2: /UART4_RX -> /I2C1_SCL
- R48 pad 1: Net-(J7-Pad2) -> OUT-
- R48 pad 2: /UART4_TX -> /LED_Capa
- R49 pad 1: Net-(Q10-D) -> /LED_Capa
- R49 pad 2: /capa_out -> Net-(Q12-G)
- R5 pad 1: /TIM1_CH1 -> Net-(SW1-B)
- R5 pad 2: -H30 -> /BOOT0
- R50 pad 1: /LED_Capa -> Net-(J9-Pad3)
- R50 pad 2: Net-(Q11-G) -> /UART4_RX
- R51 pad 1: +3V3 -> Net-(J9-Pad2)
- R51 pad 2: Net-(D13-A) -> /UART4_TX
- R53 pad 1: Net-(J8-Pad3) -> /LED_Capa
- R53 pad 2: /ADC3_IN3+ -> Net-(Q11-G)
- R54 pad 1: Net-(J8-Pad2) -> +3V3
- R54 pad 2: /ADC2_IN4 -> Net-(D14-A)
- R55 pad 1: Net-(J9-Pad3) -> Net-(Q10-D)
- R55 pad 2: /I2C1_SCA -> /capa_out
- R56 pad 1: Net-(J9-Pad2) -> Net-(J10-Pad3)
- R56 pad 2: /I2C1_SCL -> /ADC3_IN3+
- R57 pad 1: Net-(J12-Pad3) -> Net-(J10-Pad2)
- R57 pad 2: /UART5_RX -> /ADC2_IN4
- R58 pad 1: Net-(J12-Pad2) -> Net-(J11-Pad3)
- R58 pad 2: /UART5_TX -> /I2C1_SDA
- R59 pad 1: Net-(D14-K) -> Net-(J11-Pad2)
- R59 pad 2: /TIM3_CH1 -> /I2C1_SCL
- R6 pad 2: Net-(Q3-G) -> -H30
- R60 pad 1: +3V3 -> Net-(J13-Pad3)
- R60 pad 2: /ALERT1 -> /UART5_RX
- R61 pad 1: +3V3 -> Net-(J13-Pad2)
- R61 pad 2: /ALERT2 -> /UART5_TX
- R62 pad 1: +5V -> Net-(D15-K)
- R63 pad 1: /TIM3_CH1 -> +3V3
- R63 pad 2: Net-(Q14-G) -> /ALERT1
- R64 pad 1: -12V -> +3V3
- R64 pad 2: Net-(IC7-IN2-) -> /ALERT2
- R65 pad 1: Net-(IC7-IN1-) -> +5V
- R65 pad 2: Net-(IC7-OUT1) -> /TIM3_CH1
- R66 pad 1: Net-(IC7-IN2-) -> /TIM3_CH1
- R66 pad 2: /ADC2_IN4 -> Net-(Q13-G)
- R67 pad 1: +3V3 -> -12V
- R67 pad 2: /NFAULT -> Net-(IC7-IN2-)
- R68 pad 1: Net-(IC7-IN2-) -> Net-(IC7-IN1-)
- R69 pad 1: /AISEN -> Net-(IC7-IN2-)
- R69 pad 2: -H30 -> /ADC2_IN4
- R7 pad 1: +3V3 -> /TIM1_CH1
- R7 pad 2: /LED_Short -> Net-(Q2-G)
- R70 pad 1: /BISEN -> +3V3
- R70 pad 2: -H30 -> /NFAULT
- R71 pad 1: Net-(J17-Pad2) -> Net-(IC7-IN2-)
- R71 pad 2: /ADC1_EX0 -> Net-(IC7-OUT1)
- R72 pad 1: Net-(J18-Pad2) -> /AISEN
- R72 pad 2: /ADC1_EX1 -> -H30
- R73 pad 1: Net-(J19-Pad2) -> Net-(J20-Pad2)
- R73 pad 2: /ADC1_EX2 -> /ADC1_EX0
- R74 pad 1: Net-(J20-Pad2) -> Net-(J21-Pad2)
- R74 pad 2: /ADC1_EX3 -> /ADC1_EX1
- R75 pad 1: Net-(J21-Pad2) -> Net-(J22-Pad2)
- R75 pad 2: /ADC2_EX0 -> /ADC1_EX2
- R76 pad 1: Net-(J22-Pad2) -> Net-(J23-Pad2)
- R76 pad 2: /ADC2_EX1 -> /ADC1_EX3
- R77 pad 1: Net-(J23-Pad2) -> Net-(J24-Pad2)
- R77 pad 2: /ADC2_EX2 -> /ADC2_EX0
- R78 pad 1: Net-(J24-Pad2) -> Net-(J25-Pad2)
- R78 pad 2: /ADC2_EX3 -> /ADC2_EX1
- R8 pad 1: /LED_Short -> +3V3
- R8 pad 2: Net-(Q5-G) -> /LED_Short
- SW3 pad 1: Net-(D11-K) -> Net-(D12-K)
- TP1 pad 1: +VBUS -> /I2C1_SDA
- TP2 pad 1: /Gate_H30-OUT- -> /I2C1_SCL
- TP3 pad 1: /NFAULT -> /LTC gate
- U1 pad 43: unconnected-(U1-PA10-Pad43) -> /TIM1_CH3
- U1 pad 59: /I2C1_SCA -> /I2C1_SDA
Other:
- outline, holes or cut-outs redrawn

Commit message: V1.1
Parts:
- removed C31: 470 uF, Capacitor_THT_Wurth_PT:CP_Wurth_WCAP-PTHT-P5D10L12.5
- removed C33, C34, C35: 10 uF, Capacitor_SMD_Wurth:CP_Wurth_WCAP-ASLI-D4L5.5
- removed C39: C, Capacitor_SMD:C_0603_1608Metric
- removed D12: STPS2L30A, STPS2L30A:DIOM5126X265N
- removed IC7: LM358DR, LM358DR:SOIC127P600X175-8N
- removed J13: 653004114822, Connector_THT_Wurth:J_Wurth_WR-WTB_653004114822
- removed J17: 653002114822, Connector_THT_Wurth:J_Wurth_WR-WTB_653002114822
- removed R33: 10K, Resistor_SMD:R_0603_1608Metric
- removed R60, R61: 22, Resistor_SMD:R_0603_1608Metric
- removed R67: 15K, Resistor_SMD:R_0603_1608Metric
- removed R68: 220R, Resistor_SMD:R_0603_1608Metric
- removed R69: 2k2, Resistor_SMD:R_0603_1608Metric
- removed R71: 12K, Resistor_SMD:R_0603_1608Metric
- removed TP7: V_Reverse, TestPoint:TestPoint_Pad_D1.5mm
- removed U3: LTC1044, LTC1044:SOIC127P600X175-8N
- added G***: LOGO, footprints:My_robot, F.Cu at (117.8, 87.9)
- added J28: 653006114822, Connector_THT_Wurth:J_Wurth_WR-WTB_653006114822, B.Cu at (114.1, 61.2)
- added J29: Conn_02x07_Odd_Even, Connector_PinSocket_1.27mm:PinSocket_2x07_P1.27mm_Vertical, F.Cu at (138.3, 69.7)
- added J30: Conn_01x14_Socket, Connector_PinSocket_2.54mm:PinSocket_2x07_P2.54mm_Vertical, F.Cu at (134.6, 63.8)
- added R18: 2K2, Resistor_SMD:R_0603_1608Metric, F.Cu at (119.6, 63.6)
- added R19: 2K2, Resistor_SMD:R_0603_1608Metric, F.Cu at (119.6, 62.4)
- added REF**: MountingHole_2.2mm_M2_DIN965, MountingHole:MountingHole_2.2mm_M2_DIN965, B.Cu at (110.3, 62.2)
- C12: value 100nf -> 10uF; footprint Capacitor_SMD:C_0603_1608Metric -> Capacitor_SMD:C_1210_3225Metric; moved to B.Cu
- C22, C36, D16, D20, D23, D26, IC3, IC6, J20, J21, J22, J23, J24, J25, J26, J27, JP3, JP4, LS1, NT1, Q8, R31, R32, R70, R72, R81, TP4, TP8: moved to B.Cu
- J1: value XT60_YELLOW -> 662102145021; footprint XT60:AMASS_XT60PB-M -> MPC3_Wurth:J_Wurth_WR-MPC3_662102145021
- J11: value 653004114822 -> 653006114822; footprint Connector_THT_Wurth:J_Wurth_WR-WTB_653004114822 -> Connector_THT_Wurth:J_Wurth_WR-WTB_653006114822
- J18, J19: value 653002114822 -> 653102131822; footprint Connector_THT_Wurth:J_Wurth_WR-WTB_653002114822 -> Connector_SMD_Wurth:J_Wurth_WR-WTB_653102131822; moved to B.Cu
- J3: footprint Connector_PinHeader_1.27mm:PinHeader_2x07_P1.27mm_Vertical_SMD -> Connector_PinHeader_1.27mm:PinHeader_2x07_P1.27mm_Vertical
- R1, R40, R41, R42, R43, R73, R74, R75, R76, R77, R78, R79, R80: footprint Resistor_SMD:R_0603_1608Metric -> Resistor_SMD:R_0402_1005Metric
- R38, R39, R44, R45, R46, R47, R50, R51, R56, R57, R58, R59: footprint Resistor_SMD:R_0603_1608Metric -> Resistor_SMD:R_0402_1005Metric; moved to B.Cu
- R52, R55: footprint Resistor_SMD:R_0603_1608Metric -> Resistor_SMD:R_1210_3225Metric
- SW1, SW3: footprint Button_Switch_SMD:Nidec_Copal_CAS-120A -> 450404015514:450404015514
- moved H3 135.9 mm to (97.4, 78.1)
- moved C18 108.2 mm to (154.8, 88.8), turned to 90 degrees
- moved C2 106.4 mm to (150.3, 82.2)
- moved R35 105.9 mm to (161.0, 109.4)
- moved C12 105.4 mm to (152.7, 91.7), turned to 90 degrees
- moved R2 103.6 mm to (153.4, 90.2), turned to 90 degrees
- moved R11 103.1 mm to (160.2, 76.8), turned to -90 degrees
- moved R8 102.4 mm to (158.7, 79.7), turned to -90 degrees
- moved R10 102.1 mm to (158.7, 82.7), turned to -90 degrees
- moved C36 101.9 mm to (154.2, 87.2), turned to 180 degrees
- moved R6 101.7 mm to (157.3, 79.7), turned to -90 degrees
- moved R7 99.2 mm to (155.2, 79.7), turned to -90 degrees
- moved R5 98.7 mm to (153.8, 79.7), turned to -90 degrees
- moved R3 98.5 mm to (152.3, 79.7), turned to 90 degrees
- moved C13 97.5 mm to (145.7, 88.2), turned to -90 degrees
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Connections:
- C10 pad 2: -H30 -> -ST
- C12 pad 1: +3V3 -> +H30
- C12 pad 2: -ST -> -H30
- C15 pad 2: -H30 -> -ST
- C17 pad 2: -H30 -> -ST
- C24 pad 2: Net-(Q10-D) -> /capa_out
- C27 pad 2: Net-(Q10-D) -> /capa_out
- C29 pad 2: Net-(Q10-D) -> /capa_out
- C30 pad 2: Net-(Q10-D) -> /capa_out
- C32 pad 2: Net-(Q10-D) -> /capa_out
- C37 pad 1: +5V -> +3V3
- C38 pad 1: +5V -> +3V3
- C4 pad 2: -H30 -> -ST
- C6 pad 2: -H30 -> -ST
- D9 pad 1: -H30 -> -ST
- H1 pad 1: -H30 -> unconnected-(H1-Pad1)
- H2 pad 1: -H30 -> unconnected-(H2-Pad1)
- H3 pad 1: -H30 -> unconnected-(H3-Pad1)
- H4 pad 1: -H30 -> unconnected-(H4-Pad1)
- IC1 pad 4: -H30 -> -ST
- IC4 pad 8: +5V -> +3V3
- IC5 pad 1: +5V -> +3V3
- IC5 pad 8: +5V -> +3V3
- IC6 pad 12: +12V -> +H30
- J11 pad 2: Net-(J11-Pad2) -> /ALERT2
- J11 pad 3: Net-(J11-Pad3) -> /ALERT1
- J11 pad 4: +3V3 -> Net-(J11-Pad4)
- J19 pad 1: Net-(IC6-BOUT1) -> Net-(IC6-BOUT2)
- J19 pad 2: Net-(IC6-BOUT2) -> Net-(IC6-BOUT1)
- JP3 pad 2: +3V3 -> Net-(J7-Pad2)
- JP3 pad 3: Net-(J7-Pad2) -> +3V3
- JP4 pad 2: +3V3 -> Net-(J12-Pad2)
- JP4 pad 3: Net-(J12-Pad2) -> +3V3
- Q1 pad 1: -H30 -> -ST
- Q10 pad 5: Net-(Q10-D) -> /capa_out
- Q10 pad 6: (no net) -> /capa_out
- Q12 pad 1: OUT- -> /capa_out
- Q12 pad 2: OUT- -> /capa_out
- Q12 pad 3: OUT- -> /capa_out
- Q12 pad 5: /capa_out -> Net-(Q12-D)
- Q12 pad 6: (no net) -> Net-(Q12-D)
- Q4 pad 6: (no net) -> +H30
- Q5 pad 6: (no net) -> OUT+
- Q7 pad 6: (no net) -> OUT-
- R14 pad 1: -H30 -> -ST
- R17 pad 1: -H30 -> -ST
- R36 pad 1: /capa_out -> OUT+
- R52 pad 1: Net-(Q10-D) -> OUT+
- R52 pad 2: /capa_out -> Net-(Q12-D)
- R54 pad 1: +3V3 -> OUT+
- R55 pad 1: Net-(Q10-D) -> OUT+
- R55 pad 2: /capa_out -> Net-(Q12-D)
- R58 pad 1: Net-(J11-Pad3) -> Net-(J11-Pad5)
- R59 pad 1: Net-(J11-Pad2) -> Net-(J11-Pad4)
Routing:
- net -H30: track 0.00 -> 97.9 mm, vias 0 -> 32
- net +3V3: track 0.00 -> 96.0 mm, vias 0 -> 33
- net -ST: track 0.00 -> 69.1 mm, vias 0 -> 34
- net /NRST: track 0.00 -> 64.1 mm, vias 0 -> 4
- net +5V: track 0.00 -> 50.0 mm, vias 0 -> 6
- net /BIN2: track 0.00 -> 42.8 mm, vias 0 -> 1
- net +H30: track 0.00 -> 42.4 mm, vias 0 -> 3
- net /BIN1: track 0.00 -> 42.2 mm, vias 0 -> 1
- net /AIN1: track 0.00 -> 42.2 mm, vias 0 -> 1
- net Net-(D13-K): track 0.00 -> 41.4 mm, vias 0 -> 2
- net /AIN2: track 0.00 -> 41.4 mm, vias 0 -> 1
- net OUT-: track 0.00 -> 40.2 mm, vias 0 -> 37
- net /TIM1_CH1: track 0.00 -> 39.7 mm, vias 0 -> 2
- net Net-(Q9-G): track 0.00 -> 39.7 mm, vias 0 -> 2
- net /I2C1_SCL: track 0.00 -> 33.5 mm, vias 0 -> 4
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- added copper zone on B.Cu, net +3V3
- added copper zone on In2.Cu, net +3V3
- added copper zone on F.Cu, net +H30
- added copper zone on B.Cu, net -H30
- added copper zone on F.Cu, net -H30
- added copper zone on In1.Cu, net -H30
- added copper zone on In2.Cu, net -H30
- added copper zone on B.Cu, net -ST
- added copper zone on F.Cu, net -ST
- added copper zone on In1.Cu, net -ST
- added copper zone on In2.Cu, net -ST
- added copper zone on F.Cu, net /capa_out
- added copper zone on B.Cu, net OUT+
- added copper zone on F.Cu, net OUT+
- added copper zone on B.Cu, net OUT-
- added copper zone on F.Cu, net OUT-
- added copper zone on In1.Cu, net OUT-
- added copper zone on In2.Cu, net OUT-
Other:
- board size 81.2 x 116.5 mm -> 80 x 50 mm
- copper layers 2 -> 4
- board text added: "5V"
- board text added: "Arrivée cable H30 Fan"
- board text added: "BAS"
- board text added: "DFU"
- board text added: "EV"
- board text added: "HAUT"
- board text added: "PWR"
- board text added: "RST"
- board text added: "external ADC"
- board text added: "isol"

Commit message: PCB V1.1
Parts:
- C8: footprint Capacitor_SMD:C_0603_1608Metric -> Capacitor_SMD:C_0402_1005Metric
- moved J30 36.5 mm to (108.2, 38.5)
- moved J29 36.3 mm to (112.2, 44.4)
- moved C8 36.1 mm to (89.2, 55.7)
- moved Q8 36.0 mm to (100.0, 66.2)
- moved R32 36.0 mm to (100.1, 63.5)
- moved H1 35.8 mm to (138.6, 53.4)
- moved H2 35.8 mm to (140.1, 80.3)
- moved IC6 35.8 mm to (133.7, 62.6)
- moved J15 35.8 mm to (128.9, 77.5)
- moved J19 35.8 mm to (142.6, 63.6)
- moved R22 35.8 mm to (129.0, 61.1)
- moved SW1 35.8 mm to (128.2, 50.9)
- moved C18 35.8 mm to (129.0, 64.0)
- moved IC2 35.8 mm to (135.1, 80.8)
- moved J1 35.8 mm to (142.0, 62.0)
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- renumbered TP6 to -ST, TP2 to SCL, TP1 to SDA
Routing:
- net /BOOT0: track 0.00 -> 44.5 mm, vias 0 -> 2
- net /I2C1_SCL: track 33.5 -> 63.3 mm, vias 4 -> 8
- net /I2C1_SDA: track 32.6 -> 60.7 mm, vias 5 -> 8
- net -ST: track 69.1 -> 94.8 mm, vias 34 -> 43
- net /USART3_RX: track 0.00 -> 23.1 mm, vias 0 -> 2
- net /ADC1_IN1+: track 0.00 -> 20.7 mm, vias 0 -> 2
- net /USART3_TX: track 0.00 -> 20.6 mm, vias 0 -> 2
- net /SPI1_CS: track 0.00 -> 18.1 mm, vias 0 -> 2
- net /ADC3_IN3+: track 0.00 -> 17.2 mm, vias 0 -> 1
- net /SPI1_MISO: track 0.00 -> 16.7 mm, vias 0 -> 1
- net /SPI1_MOSI: track 0.00 -> 15.8 mm, vias 0 -> 1
- net /QUADSPI_NCS: track 0.00 -> 15.3 mm, vias 0 -> 1
- net /ADC1_IN2-: track 0.00 -> 14.5 mm, vias 0 -> 2
- net /UART4_RX: track 0.00 -> 13.0 mm, vias 0 -> 2
- net /14: track 17.3 -> 6.06 mm
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Other:
- outline, holes or cut-outs redrawn
- board text added: "1"
- board text added: "ADC"
- board text added: "Adapatateur 1mm 2.56mm"
- board text added: "I2C"
- board text added: "I2C & alert"
- board text added: "JTAG"
- board text added: "SPI"
- board text added: "UART"

Commit message: V1.2
Parts:
- added G***: LOGO, footprints:My_robot, B.Cu at (99.6, 82.4)
- added IC8: 114993390, 114993390:114993390, B.Cu at (105.4, 55.0)
- added JP5: ~, jumper_footprints:Jumper_3points_0402, B.Cu at (104.0, 59.2)
- renumbered SDA to TP1, SCL to TP2, -ST to TP6
Connections:
- LS1 pad 3: unconnected-(LS1-NC_1-Pad3) -> OUT+
- U1 pad 20: unconnected-(U1-PA4-Pad20) -> /SPI1_NSS
- U1 pad 28: unconnected-(U1-PB2-Pad28) -> /GPIO_BUSY
- U1 pad 33: unconnected-(U1-PB12-Pad33) -> /LORA_NRST
- U1 pad 34: unconnected-(U1-PB13-Pad34) -> /GPIO_EXTI13
Routing:
- net /SPI1_MOSI: track 15.8 -> 59.5 mm, vias 1 -> 4
- net /GPIO_BUSY: track 0.00 -> 32.6 mm, vias 0 -> 3
- net /SPI1_MISO: track 16.7 -> 46.0 mm, vias 1 -> 3
- net /SPI1_NSS: track 0.00 -> 29.1 mm, vias 0 -> 4
- net /GPIO_EXTI13: track 0.00 -> 27.8 mm, vias 0 -> 2
- net /SPI1_SCK: track 5.71 -> 30.3 mm, vias 0 -> 2
- net /LORA_NRST: track 0.00 -> 20.2 mm, vias 0 -> 3
- net OUT+: track 35.1 -> 51.5 mm
- net -ST: track 94.8 -> 101.3 mm, vias 43 -> 42
- net Net-(IC8-RF_SW_): track 0.00 -> 5.37 mm
- net +3V3: track 102.1 -> 104.1 mm, vias 33 -> 35
- net Net-(Q11-G): track 5.23 -> 6.89 mm
- net /TIM3_CH1: track 15.0 -> 16.4 mm
- net -H30: track 97.9 -> 98.9 mm
- net /NRST: track 64.0 -> 64.8 mm
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Other:
- board text added: "Controller H30 V1"
- board text added: "Maxence HEROUX Promo 2028"
- board text added: "Stetching !"
- board text added: "silckscreen + IHM !"
