File: PCB/H30_controler_board.kicad_pcb (KiCad board)
At the start: 4 copper layers, 80 x 50 mm, 216 parts, among them IC1 MP2338GTL-P, IC2 LTC4359IMS8#PBF, IC3 W25N01GVZEIG, IC4 ADS1115IDGSR, IC5 ADS1115IDGSR, IC6 DRV8833CPWPR, IC8 114993390, J1 662102145021, J10 653004114822, J11 653006114822, J12 653002114822, J14 653006114822, J15 XT60_YELLOW, J16 653002114822, J18 653102131822, J19 653102131822, J2 USB_C_Receptacle_USB2.0_14P, J20 653003114822, J21 653003114822, J22 653003114822, J23 653003114822, J24 653003114822, J25 653003114822, J26 653003114822, J27 653003114822, J28 653006114822, J29 Conn_02x07_Odd_Even, J3 SWD, J30 Conn_01x14_Socket, J4 653004114822, J5 653004114822, J6 653004114822, J7 653002114822, J8 TC2030, J9 653004114822, Q1 AO3401A, Q10 PSMNR56-25YLEX, Q11 2N7002, Q12 PSMNR56-25YLEX, Q13 SI2301-TP, Q2 SI2301-TP, Q3 2N7002, Q4 PSMNR56-25YLEX, Q5 PSMNR56-25YLEX, Q6 SI2301-TP, Q7 PSMNR56-25YLEX, Q8 2N7002, Q9 SI2301-TP, SW1 SW_Nidec_CAS-120A1, SW3 SW_Nidec_CAS-120A1, U1 STM32L476RCTx, U2 USBLC6-2SC6, Y1 16MHz

Commit message: PCB V1.2
Parts:
- moved JP5 5.31 mm to (103.8, 64.5)
- moved R31 3.23 mm to (99.1, 69.1)
Connections:
- J19 pad MP1: (no net) -> -H30
Routing:
- net -ST: track 101.3 -> 114.3 mm, vias 42 -> 51
- net Net-(IC8-RF_SW_): track 5.37 -> 16.0 mm, vias 0 -> 2
- net /capa_out: track 5.40 -> 9.85 mm
- net +3V3: track 104.1 -> 107.7 mm, vias 35 -> 36
- net Net-(LS1--): track 8.48 -> 11.7 mm
- net Net-(SW1-B): track 1.37 -> 2.84 mm
- net /LED_Capa: track 16.0 -> 16.9 mm
- net +5V: track 50.6 -> 51.5 mm
- net /SPI1_MISO: track 46.0 -> 45.2 mm
- net Net-(IC1-SS): track 2.21 -> 2.81 mm
- net -H30: track 98.9 -> 99.3 mm, vias 32 -> 36
- net OUT-: track 40.2 -> 40.6 mm, vias 37 -> 46
Other:
- board text added: "3v"
- board text added: "5v"
- board text added: "External ADC *8 (16bit)"
- board text added: "JTAG adaptateur"
- board text added: "Rx"
- board text added: "Tx"
- board text removed: "Stetching !"
- board text removed: "silckscreen + IHM !"
